File: power.sch (KiCad schematic (older format))
At the start: 83 parts, among them J1 USB_2, P1 AC, P10 CONN_2, P2 ISP, P3 CONN_2, P4 CONN_2, P5 CONN_2, P6 CONN_2, P7 CONN_2, P8 CONN_2, P9 CONN_2, Q1 BC237, T1 230V/12V, T2 BT136, T3 BT136, T4 BT136, T5 BT136, T6 BT136, T7 BT136, T8 BT136, T9 BT136, U1 FT232RL, U10 MOC3022M, U11 MOC3022M, U12 MOC3022M, U13 MOC3022M, U14 MOC3022M, U2 LM7805, U3 74LS259, U4 ATMEGA644P-P, U5 74LS04, U6 74LS04, U7 MOC3022M, U8 MOC3022M, U9 MOC3022M, X1 16MHz

Commit message: Updated schema with more complete circuit
Parts:
- removed F2: 5A, symbol FUSE_IEC
- removed P10, P4, P5, P6, P7, P8, P9: CONN_2, symbol CONN_2
- removed R10, R11, R12, R13, R7, R8, R9: 1k, symbol R_IEC
- removed T3, T4, T5, T6, T7, T8, T9: BT136, symbol TRIAC_IEC
- removed TH2, TH3, TH4, TH5, TH6, TH7, TH8: 30R500, symbol THERMISTOR
- removed U10, U11, U12, U13, U14, U8, U9: MOC3022M, DIP6, symbol MOC3022M
- removed U3: 74LS259, symbol 74LS259
- removed unit 2 of U5
- removed unit 3 of U5
- removed unit 4 of U5
- removed unit 5 of U5
- removed unit 6 of U5
- removed U6: 74LS04, symbol 74LS04
- added C? (x7): 100n, symbol C_IEC
- added C? (x7): 220n, symbol C_IEC
- added C? (x5): 1u, symbol CP_IEC
- added J?: DB9, symbol DB9
- added L? (x7): 100u, symbol L_IEC
- added P? (x7): CONN_2, symbol CONN_2
- added R? (x7): 1k, symbol R_IEC
- added R? (x14): 100, symbol R_IEC
- added R? (x7): 33, symbol R_IEC
- added T? (x7): BT136, symbol TRIAC_IEC
- added TH? (x7): 30R500, symbol THERMISTOR
- added U? (x7): 74LS04, symbol 74LS04
- added U? (x7): MOC3022M, DIP6, symbol MOC3022M
- added U?: MAX232, symbol MAX232
- F1: value 5A -> 8A
Connections:
- net labels added: M1, M2, M3, M4, M5, M6, M7, M8
- net labels removed: M1S, M2S, M3S, M4S, M5S, M6S, M7S, M8S
- wire segments 90 -> 130
Other:
- moved on the sheet: P1, P2, P3, U1, X1
