File: control.sch (KiCad schematic (older format))
At the start: 130 parts, among them IC1 TJA1040, IC2 DNP MAX481CSA, IC3 ST232BD, IC4 ATMEGA128-A, IC5 ST232BD, IC6 FT232RL, J1 DB9, J2 B, J3 USB_4, J4 POWER, J5 DB9, P1 SENSOR, P2 I2C0, P3 I2C1, P4 I2C2, P5 COIN, P6 BILL, P7 ISP, P8 CONN_2, P9 CONN_2, X1 16MHz

Commit message: Fixed a number of errata in first control board revision Swapped USB B port D+ and D- lines Swapped UART0 RX and TX lines Changed resistor values Added UART0 RX and TX LEDs Conntected USB sleep control line
Parts:
- added D4, D5: LED805, LED-0805, symbol LED
- added R68: DNP, -R2012, symbol R_IEC
- added R69, R70: 1k, -R2012, symbol R_IEC
- C24: footprint -R2012 -> C1V5
- R3: value 1k -> 0
- R5: value DNP -> 0
Connections:
- net labels added: LED RX, LED TX, USB_SLEEP
- net labels removed: USB_EN
- wire segments 290 -> 298
Other:
- moved on the sheet: C20, C23, C24, C25, C26, C27, C31, C32, D1, D2, D3, IC6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

Commit message: Added component library Updated conmponents in schematic Changed resistors and capacitors to standard symbol
Parts:
- C1, C10, C11, C12, C13, C14, C15, C16, C17, C18, C19, C2, C20, C21, C22, C23, C25, C27, C28, C29, C3, C30, C31, C4, C5, C6, C7, C8, C9: symbol C_IEC -> C
- C24, C26, C32: symbol CP_IEC -> CP1
- IC2: symbol _STO-MAX481CSA -> MAX481CSA
- J2: symbol USB_2 -> USB_B_5
- J3: symbol USB_4 -> USB_MINI_B_6
- L1: symbol L_IEC -> INDUCTOR
- R1, R10, R11, R12, R13, R14, R15, R16, R17, R18, R19, R2, R20, R21, R22, R23, R24, R25, R26, R27, R28, R29, R3, R30, R31, R32, R33, R34, R35, R36, R37, R38, R39, R4, R40, R41, R42, R43, R44, R45, R46, R47, R48, R49, R5, R50, R51, R52, R53, R54, R55, R56, R57, R58, R59, R6, R60, R61, R62, R63, R64, R65, R66, R67, R68, R69, R7, R70, R8, R9: symbol R_IEC -> R
- X1: symbol XTAL_IEC -> CRYSTAL
Connections:
- wire segments 298 -> 300
Other:
- moved on the sheet: C12, C13, C14, C15, C16, C17, C18, C19, C5, C6, J1, P1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

Commit message: Fixed banknote scanner connector erratum, short circuit on power lines
Connections:
- wire segments 300 -> 403
