File: control.sch (KiCad schematic (older format))
At the start: 135 parts, among them IC1 TJA1040, IC2 DNP MAX481CSA, IC3 ST232BD, IC4 ATMEGA128-A, IC5 ST232BD, IC6 FT232RL, J1 DB9, J2 B, J3 USB_4, J4 POWER, J5 DB9, P1 SENSOR, P2 I2C0, P3 I2C1, P4 I2C2, P5 COIN, P6 BILL, P7 ISP, P8 CONN_2, P9 CONN_2, X1 16MHz

Commit message: Added module library Fixed up schema with new part names Partial PCB redesign, incorporated schematic changes and errata Made PCB slightly smaller
Parts:
- C1, C10, C11, C12, C13, C14, C15, C16, C17, C18, C19, C2, C20, C21, C22, C23, C25, C27, C28, C29, C3, C30, C31, C4, C5, C6, C7, C8, C9, R1, R10, R11, R12, R13, R14, R15, R16, R17, R18, R19, R2, R20, R21, R22, R23, R24, R25, R26, R27, R28, R29, R3, R30, R31, R32, R33, R34, R35, R36, R37, R38, R39, R4, R40, R41, R42, R43, R44, R45, R46, R47, R48, R49, R5, R50, R51, R52, R53, R54, R55, R56, R57, R58, R59, R6, R60, R61, R62, R63, R64, R65, R66, R67, R68, R69, R7, R70, R8, R9: footprint -R2012 -> R0805
- IC4: footprint -TQFP64 -> TQFP64
- IC6: footprint -SSOP28 -> SSOP28
- J1, J5: footprint DB9MC -> DB9MCS
- J3: footprint oni_USB_MINI_B -> USB_MINI_B_6
- X1: footprint crystal-SM49 -> Q_49U3HMS
Connections:
- wire segments 403 -> 296

Commit message: Updated PCB Placed part labels Moved some parts to use space more efficiently
Parts:
- renumbered J1 to P10, J2 to P11, J3 to P12, J5 to P13
Changed lines of the file:
@@
 Sheet 1 1
 Title "Matemat Control Circuit"
-Date "5 apr 2015"
+Date "6 apr 2015"
 Rev "5"
 Comp "Chaostreff Basel"
@@
 $EndComp
 $Comp
-L DB9 J5
+L DB9 P13
 U 1 1 50A30577
 P 15650 5200
-F 0 "J5" H 15650 5750 70  0000 C CNN
+F 0 "P13" H 15650 5750 70  0000 C CNN
 F 1 "DB9" H 15650 4650 70  0000 C CNN
 F 2 "DB9MCS" H 15650 5200 60  0001 C CNN
@@
 $EndComp
 $Comp
-L DB9 J1
+L DB9 P10
 U 1 1 5116C3F6
 P 5650 9950
-F 0 "J1" H 5650 10500 70  0000 C CNN
+F 0 "P10" H 5650 10500 70  0000 C CNN
 F 1 "DB9" H 5650 9400 70  0000 C CNN
 F 2 "DB9MCS" H 5650 9950 60  0001 C CNN
@@
 $EndComp
 $Comp
-L USB_MINI_B_6 J3
+L USB_MINI_B_6 P12
 U 1 1 51522CC2
 P 11600 2650
-F 0 "J3" H 11500 2300 60  0000 C CNN
+F 0 "P12" H 11500 2300 60  0000 C CNN
 F 1 "USB_4" H 11650 2300 60  0001 C CNN
 F 2 "USB_MINI_B_6" H 11600 2650 60  0001 C CNN
@@
 $EndComp
 $Comp
-L USB_B_5 J2
+L USB_B_5 P11
 U 1 1 51522D4C
 P 11600 2000
-F 0 "J2" H 11500 2300 60  0000 C CNN
+F 0 "P11" H 11500 2300 60  0000 C CNN
 F 1 "B" V 11500 2150 60  0000 C CNN
 F 2 "USB_B" H 11600 2000 60  0001 C CNN
