File: control.kicad_pcb (KiCad board)
At the start: 2 copper layers, 140 x 103.2 mm, 135 parts, among them IC1 TJA1040, IC2 MAX481, IC3 ST232BD, IC4 ATMEGA128-A, IC5 ST232BD, IC6 FT232RL, J4 POWER, P1 SENSOR, P10 DB9, P11 USB_B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

Commit message: Added copyright field and OSHW logo to PCB
Parts:
- added SYM: Symbol_OSHW-Logo_SilkScreen_07Jul2012, Symbol_OSHW-Logo_SilkScreen_07Jul2012, F.Cu at (55.0, 143.6)
Other:
- board text added: "Matemat Controller © 2015 Chaostreff Basel Revision 4"
