File: control/control.sch (KiCad schematic (older format))
At the start: 136 parts, among them IC1 TJA1040, IC2 DNP MAX481CSA, IC3 ST232BD, IC4 ATMEGA128-A, IC5 ST232BD, IC6 FT232RL, J4 POWER, P1 SENSOR, P10 DB9, P11 USB_B, P12 USB_OTG, P13 DB9, P2 I2C0, P3 I2C1, P4 I2C2, P5 COIN, P6 CONN_02X13, P7 ISP, P8 12V, P9 5V, U1 DNP LM2940-N 5V, X1 16MHz

Commit message: Update and cleanup for KiCAD 5
Parts:
- C1, C10, C11, C12, C13, C14, C15, C16, C17, C18, C19, C2, C20, C21, C22, C23, C25, C27, C28, C29, C3, C30, C31, C33, C4, C5, C6, C7, C8, C9: symbol C -> control-rescue:C
- C24, C26, C32: symbol CP -> control-rescue:CP
- D1, D2, D3, D4, D5: symbol LED -> control-rescue:LED
- IC1: symbol TJA1040 -> matemat:TJA1040
- IC2: symbol MAX481CSA -> matemat:MAX481CSA
- IC3, IC5: symbol MAX232 -> control-rescue:MAX232
- IC4: symbol ATMEGA128-A -> control-rescue:ATMEGA128-A
- IC6: symbol FT232RL -> control-rescue:FT232RL
- J4: symbol Bus_I2C -> matemat:Bus_I2C
- JP1: symbol JUMPER3 -> control-rescue:JUMPER3
- JP2: symbol JUMPER -> control-rescue:JUMPER
- L1: symbol INDUCTOR -> control-rescue:INDUCTOR
- P1: symbol CONN_02X08 -> control-rescue:CONN_02X08
- P10, P13: symbol DB9 -> control-rescue:DB9
- P11: symbol USB_B -> control-rescue:USB_B
- P12: symbol USB_OTG -> control-rescue:USB_OTG
- P2, P3, P4: symbol CONN_02X05 -> control-rescue:CONN_02X05
- P5: symbol CONN_01X17 -> control-rescue:CONN_01X17
- P6: symbol CONN_02X13 -> control-rescue:CONN_02X13
- P7: symbol CONN_02X03 -> control-rescue:CONN_02X03
- P8, P9: symbol CONN_01X02 -> control-rescue:CONN_01X02
- R1, R10, R11, R12, R13, R14, R15, R16, R17, R18, R19, R2, R20, R21, R22, R23, R24, R25, R26, R27, R28, R29, R3, R30, R31, R32, R33, R34, R35, R36, R37, R38, R39, R4, R40, R41, R42, R43, R44, R45, R46, R47, R48, R49, R5, R50, R51, R52, R53, R54, R55, R56, R58, R6, R60, R61, R62, R63, R64, R65, R66, R67, R68, R69, R7, R70, R71, R8, R9: symbol R -> control-rescue:R
- TP1, TP2, TP3, TP4: symbol CONN_01X01 -> control-rescue:CONN_01X01
- U1: symbol LM2937 -> matemat:LM2937
- X1: symbol Crystal -> control-rescue:Crystal
