File: poweriface/poweriface.sch (KiCad schematic (older format))
At the start: 20 parts, among them J1 Power Board, J2 CAN In, J3 CAN Out, J4 AVR-ISP-6, U1 ATmega32M1-AU, U2 MCP2551-I-SN, Y1 16MHz

Commit message: Connected hispeed control to GPIO pin
Parts:
- added R?: 0, Resistor_SMD:R_0805_2012Metric_Pad1.15x1.40mm_HandSolder, symbol Device:R
Connections:
- net HISPEED: now reaches U1.14 (PD6)
- net HISPEED: now also R?.1
- net at R6.2, U2.8 (Rs): now also R?.2
Changed lines of the file:
@@
 EESchema Schematic File Version 4
+LIBS:poweriface-cache
 EELAYER 26 0
 EELAYER END
@@
 	7600 5500 8000 5500
 Connection ~ 7600 5500
+$Comp
+L Device:R R?
+U 1 1 5CA5C44B
+P 6200 4950
+F 0 "R?" V 6407 4950 50  0000 C CNN
+F 1 "0" V 6316 4950 50  0000 C CNN
+F 2 "Resistor_SMD:R_0805_2012Metric_Pad1.15x1.40mm_HandSolder" V 6130 4950 50  0001 C CNN
+F 3 "~" H 6200 4950 50  0001 C CNN
+	1    6200 4950
+	0    -1   -1   0
+$EndComp
+Wire Wire Line
+	6350 4950 6350 4800
+Connection ~ 6350 4800
+Text Label 6050 4950 2    50   ~ 0
+HISPEED
+Text Label 4900 3800 0    50   ~ 0
+HISPEED
+Text Label 4550 4900 0    50   ~ 0
+HISPEED
 $EndSCHEMATC

Commit message: Fixed small power plane issues
Parts:
- gave numbers to parts that had none: 1
Changed lines of the file:
@@
 Connection ~ 7600 5500
 $Comp
-L Device:R R?
+L Device:R R7
 U 1 1 5CA5C44B
 P 6200 4950
-F 0 "R?" V 6407 4950 50  0000 C CNN
+F 0 "R7" V 6407 4950 50  0000 C CNN
 F 1 "0" V 6316 4950 50  0000 C CNN
 F 2 "Resistor_SMD:R_0805_2012Metric_Pad1.15x1.40mm_HandSolder" V 6130 4950 50  0001 C CNN
