File: poweriface/poweriface.sch (KiCad schematic (older format))
At the start: 21 parts, among them J1 Power Board, J2 CAN In, J3 CAN Out, J4 AVR-ISP-6, U1 ATmega32M1-AU, U2 MCP2551-I-SN, Y1 16MHz

Commit message: Replaced crystal footprint with less wasteful one
Parts:
- Y1: footprint Crystal:Crystal_SMD_HC49-SD_HandSoldering -> Crystal:Crystal_SMD_HC49-SD
Changed lines of the file:
@@
 F 0 "Y1" V 4754 5581 50  0000 L CNN
 F 1 "16MHz" V 4845 5581 50  0000 L CNN
-F 2 "Crystal:Crystal_SMD_HC49-SD_HandSoldering" H 4800 5450 50  0001 C CNN
+F 2 "Crystal:Crystal_SMD_HC49-SD" H 4800 5450 50  0001 C CNN
 F 3 "~" H 4800 5450 50  0001 C CNN
 	1    4800 5450

Commit message: Added ground terminals
Parts:
- removed C3: 10u, Capacitor_THT:CP_Radial_D5.0mm_P2.00mm, symbol Device:CP
- removed J3: CAN Out, TerminalBlock_TE-Connectivity:TerminalBlock_TE_282834-2_1x02_P2.54mm_Horizontal, symbol Connector_Generic:Conn_01x02
- added C3: 10u, Capacitor_SMD:C_0805_2012Metric_Pad1.15x1.40mm_HandSolder, symbol Device:C
- added J3: CAN_SHIELD, TerminalBlock_TE-Connectivity:TerminalBlock_TE_282834-6_1x06_P2.54mm_Horizontal, symbol Connector_Generic:Conn_01x06
- J2: value CAN In -> CAN; footprint TerminalBlock_TE-Connectivity:TerminalBlock_TE_282834-2_1x02_P2.54mm_Horizontal -> TerminalBlock_TE-Connectivity:TerminalBlock_TE_282834-4_1x04_P2.54mm_Horizontal; symbol Connector_Generic:Conn_01x02 -> Connector_Generic:Conn_01x04
- R7: value 0 -> DNP
Connections:
- net +5V: now also C3.1
- net CAN_N: now also J2.1 (Pin_1), J2.4 (Pin_4), J3.2 (Pin_2), J3.5 (Pin_5); no longer J2.2 (Pin_2)
- net CAN_P: now also J2.2 (Pin_2), J2.3 (Pin_3), J3.3 (Pin_3), J3.4 (Pin_4); no longer J2.1 (Pin_1)
- net GND: now also C3.2, J3.1 (Pin_1), J3.6 (Pin_6)
Changed lines of the file:
@@
 EESchema Schematic File Version 4
-LIBS:poweriface-cache
-EELAYER 26 0
+EELAYER 30 0
 EELAYER END
 $Descr A4 11693 8268
@@
 Sheet 1 1
 Title "Matemat Power Board CAN Interface"
-Date "2019-04-05"
-Rev "1"
+Date "2020-02-12"
+Rev "2"
 Comp "CCC Basel"
 Comment1 ""
@@
 $EndComp
 $Comp
-L Connector_Generic:Conn_01x02 J2
-U 1 1 5CA53A5C
-P 8400 4400
-F 0 "J2" H 8479 4392 50  0000 L CNN
-F 1 "CAN In" H 8479 4301 50  0000 L CNN
-F 2 "TerminalBlock_TE-Connectivity:TerminalBlock_TE_282834-2_1x02_P2.54mm_Horizontal" H 8400 4400 50  0001 C CNN
-F 3 "~" H 8400 4400 50  0001 C CNN
-	1    8400 4400
-	1    0    0    -1
-$EndComp
-$Comp
-L Connector_Generic:Conn_01x02 J3
-U 1 1 5CA53AD4
-P 8400 4800
-F 0 "J3" H 8479 4792 50  0000 L CNN
-F 1 "CAN Out" H 8479 4701 50  0000 L CNN
-F 2 "TerminalBlock_TE-Connectivity:TerminalBlock_TE_282834-2_1x02_P2.54mm_Horizontal" H 8400 4800 50  0001 C CNN
-F 3 "~" H 8400 4800 50  0001 C CNN
-	1    8400 4800
-	1    0    0    -1
-$EndComp
-$Comp
 L Device:Crystal Y1
 U 1 1 5CA53BA3
@@
 	0    1    1    0
 $EndComp
+Text Label 8200 4600 2    50   ~ 0
+CAN_N
 Text Label 8200 4500 2    50   ~ 0
-CAN_N
-Text Label 8200 4400 2    50   ~ 0
 CAN_P
-Text Label 8200 4800 2    50   ~ 0
-CAN_P
-Text Label 8200 4900 2    50   ~ 0
-CAN_N
 Text Label 7350 4700 0    50   ~ 0
 CAN_N
@@
 Text Label 6350 4400 2    50   ~ 0
 TXCAN
-$Comp
-L Device:CP C3
-U 1 1 5CA54AD7
-P 6800 5650
-F 0 "C3" H 6918 5696 50  0000 L CNN
-F 1 "10u" H 6918 5605 50  0000 L CNN
-F 2 "Capacitor_THT:CP_Radial_D5.0mm_P2.00mm" H 6838 5500 50  0001 C CNN
-F 3 "~" H 6800 5650 50  0001 C CNN
-	1    6800 5650
-	1    0    0    -1
-$EndComp
 Wire Wire Line
 	7200 5500 6800 5500
@@
 P 6200 4950
 F 0 "R7" V 6407 4950 50  0000 C CNN
-F 1 "0" V 6316 4950 50  0000 C CNN
+F 1 "DNP" V 6316 4950 50  0000 C CNN
 F 2 "Resistor_SMD:R_0805_2012Metric_Pad1.15x1.40mm_HandSolder" V 6130 4950 50  0001 C CNN
 F 3 "~" H 6200 4950 50  0001 C CNN
@@
 Text Label 4550 4900 0    50   ~ 0
 HISPEED
+$Comp
+L Device:C C3
+U 1 1 5E445A5C
+P 6800 5650
+F 0 "C3" H 6915 5696 50  0000 L CNN
+F 1 "10u" H 6915 5605 50  0000 L CNN
+F 2 "Capacitor_SMD:C_0805_2012Metric_Pad1.15x1.40mm_HandSolder" H 6838 5500 50  0001 C CNN
+F 3 "~" H 6800 5650 50  0001 C CNN
+	1    6800 5650
+	1    0    0    -1
+$EndComp
+$Comp
+L Connector_Generic:Conn_01x04 J2
+U 1 1 5CA53A5C
+P 8400 4400
+F 0 "J2" H 8479 4392 50  0000 L CNN
+F 1 "CAN" H 8479 4301 50  0000 L CNN
+F 2 "TerminalBlock_TE-Connectivity:TerminalBlock_TE_282834-4_1x04_P2.54mm_Horizontal" H 8400 4400 50  0001 C CNN
+F 3 "~" H 8400 4400 50  0001 C CNN
+	1    8400 4400
+	1    0    0    -1
+$EndComp
+Text Label 8200 4300 2    50   ~ 0
+CAN_N
+Text Label 8200 4400 2    50   ~ 0
+CAN_P
+$Comp
+L Connector_Generic:Conn_01x06 J3
+U 1 1 5F01B6DF
+P 9200 4400
+F 0 "J3" H 9280 4392 50  0000 L CNN
+F 1 "CAN_SHIELD" H 9280 4301 50  0000 L CNN
+F 2 "TerminalBlock_TE-Connectivity:TerminalBlock_TE_282834-6_1x06_P2.54mm_Horizontal" H 9200 4400 50  0001 C CNN
+F 3 "~" H 9200 4400 50  0001 C CNN
+	1    9200 4400
+	1    0    0    -1
+$EndComp
+Text Label 9000 4600 2    50   ~ 0
+CAN_N
+Text Label 9000 4500 2    50   ~ 0
+CAN_P
+Text Label 9000 4300 2    50   ~ 0
+CAN_N
+Text Label 9000 4400 2    50   ~ 0
+CAN_P
+$Comp
+L power:GND #PWR0101
+U 1 1 5F01D002
+P 9000 4700
+F 0 "#PWR0101" H 9000 4450 50  0001 C CNN
+F 1 "GND" H 9005 4527 50  0000 C CNN
+F 2 "" H 9000 4700 50  0001 C CNN
+F 3 "" H 9000 4700 50  0001 C CNN
+	1    9000 4700
+	0    1    1    0
+$EndComp
+$Comp
+L power:GND #PWR0102
+U 1 1 5F01D90A
+P 9000 4200
+F 0 "#PWR0102" H 9000 3950 50  0001 C CNN
+F 1 "GND" H 9005 4027 50  0000 C CNN
+F 2 "" H 9000 4200 50  0001 C CNN
+F 3 "" H 9000 4200 50  0001 C CNN
+	1    9000 4200
+	0    1    1    0
+$EndComp
 $EndSCHEMATC
