File: power/matemat_power.sch (KiCad schematic (older format))
At the start: 10 parts, among them J1 B3_Wago, J2 B3_Wago, J3 B3_Wago

Commit message: Updated power board for KiCAD 5
Parts:
- F1, F2: symbol FUSE -> matemat_power-rescue:FUSE
- J1, J2, J3: symbol CONN_2 -> matemat_power-rescue:CONN_2
- TROU1, TROU2, TROU3, TROU4, TROU5: symbol CONNECTOR -> matemat_power-rescue:CONNECTOR
Connections:
- wire segments 16 -> 19
Changed lines of the file:
@@
-EESchema Schematic File Version 2
-LIBS:power
-LIBS:device
-LIBS:transistors
-LIBS:conn
-LIBS:linear
-LIBS:regul
-LIBS:74xx
-LIBS:cmos4000
-LIBS:adc-dac
-LIBS:memory
-LIBS:xilinx
-LIBS:special
-LIBS:microcontrollers
-LIBS:dsp
-LIBS:microchip
-LIBS:analog_switches
-LIBS:motorola
-LIBS:texas
-LIBS:intel
-LIBS:audio
-LIBS:interface
-LIBS:digital-audio
-LIBS:philips
-LIBS:display
-LIBS:cypress
-LIBS:siliconi
-LIBS:opto
-LIBS:atmel
-LIBS:contrib
-LIBS:valves
-LIBS:sto
-LIBS:sto2
-LIBS:40xx
-LIBS:uln-udn
-LIBS:optocoupler
-LIBS:diode-1_corr
+EESchema Schematic File Version 4
 LIBS:matemat_power-cache
-EELAYER 27 0
+EELAYER 26 0
 EELAYER END
 $Descr A4 11693 8268
@@
 $EndSheet
 $Comp
-L CONN_2 J1
+L matemat_power-rescue:CONN_2 J1
 U 1 1 50FF19C8
 P 3400 1950
@@
 $EndComp
 $Comp
-L FUSE F1
+L matemat_power-rescue:FUSE F1
 U 1 1 50FF19CE
 P 4100 2050
@@
 $EndComp
 $Comp
-L GNDPWR #PWR2
+L matemat_power-rescue:GNDPWR #PWR2
 U 1 1 50FF19D4
 P 4700 2250
@@
 	3750 2050 3850 2050
 $Comp
-L HT #PWR1
+L matemat_power-rescue:HT #PWR1
 U 1 1 50FF19DD
 P 4700 1800
@@
 $EndComp
 $Comp
-L CONN_2 J2
+L matemat_power-rescue:CONN_2 J2
 U 1 1 50FF2514
 P 3400 1500
@@
 	3750 1600 4400 1600
 Wire Wire Line
-	3750 1850 4700 1850
+	3750 1850 4500 1850
 Wire Wire Line
 	4700 1850 4700 1800
 Wire Wire Line
-	4350 2050 4700 2050
+	4350 2050 4400 2050
 Wire Wire Line
 	4700 2050 4700 2250
@@
 Connection ~ 4500 1850
 $Comp
-L CONN_2 J3
+L matemat_power-rescue:CONN_2 J3
 U 1 1 50FF3A33
 P 3400 2900
@@
 $EndComp
 $Comp
-L FUSE F2
+L matemat_power-rescue:FUSE F2
 U 1 1 50FF3A39
 P 4100 3000
@@
 $EndComp
 $Comp
-L GNDPWR #PWR4
+L matemat_power-rescue:GNDPWR #PWR4
 U 1 1 50FF3A3F
 P 4700 3200
@@
 $EndComp
 Wire Wire Line
-	3750 3000 3850 3000
-$Comp
-L HT #PWR3
+	3750 3000 3800 3000
+$Comp
+L matemat_power-rescue:HT #PWR3
 U 1 1 50FF3A46
 P 4700 2750
@@
 Connection ~ 3800 3000
 $Comp
-L CONNECTOR TROU1
+L matemat_power-rescue:CONNECTOR TROU1
 U 1 1 511ADD13
 P 8200 2250
@@
 $EndComp
 $Comp
-L CONNECTOR TROU2
+L matemat_power-rescue:CONNECTOR TROU2
 U 1 1 511ADD19
 P 8650 2250
@@
 $EndComp
 $Comp
-L CONNECTOR TROU3
+L matemat_power-rescue:CONNECTOR TROU3
 U 1 1 511ADD1F
 P 9100 2250
@@
 $EndComp
 $Comp
-L CONNECTOR TROU4
+L matemat_power-rescue:CONNECTOR TROU4
 U 1 1 511ADD25
 P 9550 2250
@@
 $EndComp
 $Comp
-L CONNECTOR TROU5
+L matemat_power-rescue:CONNECTOR TROU5
 U 1 1 511AC93D
 P 9950 2250
@@
 	0    1    1    0
 $EndComp
+Wire Wire Line
+	4400 2050 4700 2050
+Wire Wire Line
+	4500 1850 4700 1850
+Wire Wire Line
+	3800 3000 3850 3000
 $EndSCHEMATC

Commit message: Recreated rescue library
Parts:
- F1, F2: symbol matemat_power-rescue:FUSE -> matemat_power-rescue:FUSE-matemat_power-rescue
- J1, J2, J3: symbol matemat_power-rescue:CONN_2 -> matemat_power-rescue:CONN_2-matemat_power-rescue
- TROU1, TROU2, TROU3, TROU4, TROU5: symbol matemat_power-rescue:CONNECTOR -> matemat_power-rescue:CONNECTOR-matemat_power-rescue
Changed lines of the file:
@@
 EESchema Schematic File Version 4
-LIBS:matemat_power-cache
-EELAYER 26 0
+EELAYER 30 0
 EELAYER END
 $Descr A4 11693 8268
@@
 $EndSheet
 $Comp
-L matemat_power-rescue:CONN_2 J1
+L matemat_power-rescue:CONN_2-matemat_power-rescue J1
 U 1 1 50FF19C8
 P 3400 1950
@@
 $EndComp
 $Comp
-L matemat_power-rescue:FUSE F1
+L matemat_power-rescue:FUSE-matemat_power-rescue F1
 U 1 1 50FF19CE
 P 4100 2050
@@
 $EndComp
 $Comp
-L matemat_power-rescue:GNDPWR #PWR2
+L matemat_power-rescue:GNDPWR-matemat_power-rescue #PWR2
 U 1 1 50FF19D4
 P 4700 2250
@@
 	3750 2050 3850 2050
 $Comp
-L matemat_power-rescue:HT #PWR1
+L matemat_power-rescue:HT-matemat_power-rescue #PWR1
 U 1 1 50FF19DD
 P 4700 1800
@@
 $EndComp
 $Comp
-L matemat_power-rescue:CONN_2 J2
+L matemat_power-rescue:CONN_2-matemat_power-rescue J2
 U 1 1 50FF2514
 P 3400 1500
@@
 Connection ~ 4500 1850
 $Comp
-L matemat_power-rescue:CONN_2 J3
+L matemat_power-rescue:CONN_2-matemat_power-rescue J3
 U 1 1 50FF3A33
 P 3400 2900
@@
 $EndComp
 $Comp
-L matemat_power-rescue:FUSE F2
+L matemat_power-rescue:FUSE-matemat_power-rescue F2
 U 1 1 50FF3A39
 P 4100 3000
@@
 $EndComp
 $Comp
-L matemat_power-rescue:GNDPWR #PWR4
+L matemat_power-rescue:GNDPWR-matemat_power-rescue #PWR4
 U 1 1 50FF3A3F
 P 4700 3200
@@
 	3750 3000 3800 3000
 $Comp
-L matemat_power-rescue:HT #PWR3
+L matemat_power-rescue:HT-matemat_power-rescue #PWR3
 U 1 1 50FF3A46
 P 4700 2750
@@
 Connection ~ 3800 3000
 $Comp
-L matemat_power-rescue:CONNECTOR TROU1
+L matemat_power-rescue:CONNECTOR-matemat_power-rescue TROU1
 U 1 1 511ADD13
 P 8200 2250
@@
 $EndComp
 $Comp
-L matemat_power-rescue:CONNECTOR TROU2
+L matemat_power-rescue:CONNECTOR-matemat_power-rescue TROU2
 U 1 1 511ADD19
 P 8650 2250
@@
 $EndComp
 $Comp
-L matemat_power-rescue:CONNECTOR TROU3
+L matemat_power-rescue:CONNECTOR-matemat_power-rescue TROU3
 U 1 1 511ADD1F
 P 9100 2250
@@
 $EndComp
 $Comp
-L matemat_power-rescue:CONNECTOR TROU4
+L matemat_power-rescue:CONNECTOR-matemat_power-rescue TROU4
 U 1 1 511ADD25
 P 9550 2250
@@
 $EndComp
 $Comp
-L matemat_power-rescue:CONNECTOR TROU5
+L matemat_power-rescue:CONNECTOR-matemat_power-rescue TROU5
 U 1 1 511AC93D
 P 9950 2250

Commit message: Cleaned up schematics and removed obsolete parts
Parts:
- F1, F2: footprint FUSE5-20 -> Fuse:Fuseholder_Cylinder-5x20mm_Schurter_0031_8201_Horizontal_Open; symbol matemat_power-rescue:FUSE-matemat_power-rescue -> Device:Fuse
- J1, J2, J3: footprint Bornier_B2_Wago -> TerminalBlock_WAGO:TerminalBlock_WAGO_236-102_1x02_P5.00mm_45Degree; symbol matemat_power-rescue:CONN_2-matemat_power-rescue -> Connector_Generic:Conn_01x02
- TROU1, TROU2, TROU3, TROU4, TROU5: footprint TROU3 -> MountingHole:MountingHole_3.2mm_M3; symbol matemat_power-rescue:CONNECTOR-matemat_power-rescue -> Mechanical:MountingHole
Connections:
- net at J1.1 (Pin_1): now also F1.2; no longer F1.1
- removed net GNDPWR: F1.2, F2.2, J2.1 (P1)
- net GNDPWR2 renamed AC
- net AC: now also F2.2; no longer F2.1
- net HT renamed LINE
- new net NEUT: F1.1, F2.1, J2.1 (Pin_1)

Commit message: Updated PCB layout
Parts:
- J1, J2, J3: footprint TerminalBlock_WAGO:TerminalBlock_WAGO_236-102_1x02_P5.00mm_45Degree -> TerminalBlock_WAGO:TerminalBlock_WAGO_236-402_1x02_P5.00mm_45Degree
Changed lines of the file:
@@
 F 0 "J1" V 3500 1950 50  0000 C CNN
 F 1 "B3_Wago" V 3600 1950 40  0000 C CNN
-F 2 "TerminalBlock_WAGO:TerminalBlock_WAGO_236-102_1x02_P5.00mm_45Degree" H 3550 1950 60  0001 C CNN
+F 2 "TerminalBlock_WAGO:TerminalBlock_WAGO_236-402_1x02_P5.00mm_45Degree" H 3550 1950 60  0001 C CNN
 F 3 "" H 3550 1950 60  0001 C CNN
 F 4 "FAR 1283527" H 3550 1950 60  0001 C CNN "Reference"
@@
 F 0 "J2" V 3500 1600 50  0000 C CNN
 F 1 "B3_Wago" V 3600 1600 40  0000 C CNN
-F 2 "TerminalBlock_WAGO:TerminalBlock_WAGO_236-102_1x02_P5.00mm_45Degree" H 3550 1600 60  0001 C CNN
+F 2 "TerminalBlock_WAGO:TerminalBlock_WAGO_236-402_1x02_P5.00mm_45Degree" H 3550 1600 60  0001 C CNN
 F 3 "" H 3550 1600 60  0001 C CNN
 F 4 "FAR 1283527" H 3550 1600 60  0001 C CNN "Reference"
@@
 F 0 "J3" V 3500 3000 50  0000 C CNN
 F 1 "B3_Wago" V 3600 3000 40  0000 C CNN
-F 2 "TerminalBlock_WAGO:TerminalBlock_WAGO_236-102_1x02_P5.00mm_45Degree" H 3550 3000 60  0001 C CNN
+F 2 "TerminalBlock_WAGO:TerminalBlock_WAGO_236-402_1x02_P5.00mm_45Degree" H 3550 3000 60  0001 C CNN
 F 3 "" H 3550 3000 60  0001 C CNN
 F 4 "FAR 1283527" H 3550 3000 60  0001 C CNN "Reference"
