File: power/triac_channel_1.sch (KiCad schematic (older format))
At the start: 11 parts, among them J101 Output, T101 BT136, U101 MOC3022M

Commit message: Updated power board for KiCAD 5
Parts:
- C101, C102, C103: symbol C -> matemat_power-rescue:C
- J101: symbol CONN_2 -> matemat_power-rescue:CONN_2
- R101, R102, R103, R104, R105: symbol R -> matemat_power-rescue:R
- T101: symbol TRIAC_IEC -> matemat_power-rescue:TRIAC_IEC
- U101: symbol MOC3022M -> matemat_power-rescue:MOC3022M
Changed lines of the file:
@@
-EESchema Schematic File Version 2
-LIBS:power
-LIBS:device
-LIBS:transistors
-LIBS:conn
-LIBS:linear
-LIBS:regul
-LIBS:74xx
-LIBS:cmos4000
-LIBS:adc-dac
-LIBS:memory
-LIBS:xilinx
-LIBS:special
-LIBS:microcontrollers
-LIBS:dsp
-LIBS:microchip
-LIBS:analog_switches
-LIBS:motorola
-LIBS:texas
-LIBS:intel
-LIBS:audio
-LIBS:interface
-LIBS:digital-audio
-LIBS:philips
-LIBS:display
-LIBS:cypress
-LIBS:siliconi
-LIBS:opto
-LIBS:atmel
-LIBS:contrib
-LIBS:valves
-LIBS:sto
-LIBS:sto2
-LIBS:40xx
-LIBS:uln-udn
-LIBS:optocoupler
-LIBS:diode-1_corr
+EESchema Schematic File Version 4
 LIBS:matemat_power-cache
-EELAYER 27 0
+EELAYER 26 0
 EELAYER END
 $Descr A4 11693 8268
@@
 $EndDescr
 $Comp
-L MOC3022M U101
+L matemat_power-rescue:MOC3022M U101
 U 1 1 50FB1912
 P 4200 4550
@@
 $EndComp
 $Comp
-L R R101
+L matemat_power-rescue:R R101
 U 1 1 50FB1948
 P 3850 4100
@@
 $EndComp
 $Comp
-L R R103
+L matemat_power-rescue:R R103
 U 1 1 50FB1B13
 P 5600 3850
@@
 $EndComp
 $Comp
-L R R104
+L matemat_power-rescue:R R104
 U 1 1 50FB1B1E
 P 6450 4200
@@
 $EndComp
 $Comp
-L R R105
+L matemat_power-rescue:R R105
 U 1 1 50FB1B29
 P 5600 4950
@@
 $EndComp
 $Comp
-L C C101
+L matemat_power-rescue:C C101
 U 1 1 50FB1C81
 P 5250 4200
@@
 $EndComp
 $Comp
-L R R102
+L matemat_power-rescue:R R102
 U 1 1 50FB1CF2
 P 4950 4650
@@
 $EndComp
 $Comp
-L TRIAC_IEC T101
+L matemat_power-rescue:TRIAC_IEC T101
 U 1 1 50FB18FA
 P 5950 4550
@@
 $EndComp
 $Comp
-L GNDPWR #PWR01
+L matemat_power-rescue:GNDPWR #PWR01
 U 1 1 50FB1E40
 P 5250 4450
@@
 	5250 4450 5250 4400
 $Comp
-L GNDPWR #PWR02
+L matemat_power-rescue:GNDPWR #PWR02
 U 1 1 50FB1EFA
 P 5950 5250
@@
 	5950 5250 5950 4750
 $Comp
-L GNDPWR #PWR03
+L matemat_power-rescue:GNDPWR #PWR03
 U 1 1 50FB1F9D
 P 5600 5250
@@
 	5600 5250 5600 5200
 $Comp
-L GNDPWR #PWR04
+L matemat_power-rescue:GNDPWR #PWR04
 U 1 1 50FB1FD5
 P 6450 5250
@@
 	6450 4950 6450 5250
 $Comp
-L C C102
+L matemat_power-rescue:C C102
 U 1 1 50FB21D6
 P 6450 4750
@@
 $EndComp
 $Comp
-L CONN_2 J101
+L matemat_power-rescue:CONN_2 J101
 U 1 1 50FB21F2
 P 6300 3350
@@
 $EndComp
 $Comp
-L HT #PWR05
+L matemat_power-rescue:HT #PWR05
 U 1 1 50FB22BF
 P 5950 2950
@@
 	3850 4850 3850 4650
 $Comp
-L GND #PWR06
+L matemat_power-rescue:GND #PWR06
 U 1 1 50FB2A82
 P 3850 4850
@@
 $EndComp
 $Comp
-L C C103
+L matemat_power-rescue:C C103
 U 1 1 50FB266D
 P 6900 4750

Commit message: Recreated rescue library
Parts:
- C101, C102, C103: symbol matemat_power-rescue:C -> matemat_power-rescue:C-matemat_power-rescue
- J101: symbol matemat_power-rescue:CONN_2 -> matemat_power-rescue:CONN_2-matemat_power-rescue
- R101, R102, R103, R104, R105: symbol matemat_power-rescue:R -> matemat_power-rescue:R-matemat_power-rescue
- T101: symbol matemat_power-rescue:TRIAC_IEC -> matemat_power-rescue:TRIAC_IEC-matemat_power-rescue
- U101: symbol matemat_power-rescue:MOC3022M -> matemat_power-rescue:MOC3022M-matemat_power-rescue
Changed lines of the file:
@@
 EESchema Schematic File Version 4
-LIBS:matemat_power-cache
-EELAYER 26 0
+EELAYER 30 0
 EELAYER END
 $Descr A4 11693 8268
@@
 $EndDescr
 $Comp
-L matemat_power-rescue:MOC3022M U101
+L matemat_power-rescue:MOC3022M-matemat_power-rescue U101
 U 1 1 50FB1912
 P 4200 4550
@@
 $EndComp
 $Comp
-L matemat_power-rescue:R R101
+L matemat_power-rescue:R-matemat_power-rescue R101
 U 1 1 50FB1948
 P 3850 4100
@@
 $EndComp
 $Comp
-L matemat_power-rescue:R R103
+L matemat_power-rescue:R-matemat_power-rescue R103
 U 1 1 50FB1B13
 P 5600 3850
@@
 $EndComp
 $Comp
-L matemat_power-rescue:R R104
+L matemat_power-rescue:R-matemat_power-rescue R104
 U 1 1 50FB1B1E
 P 6450 4200
@@
 $EndComp
 $Comp
-L matemat_power-rescue:R R105
+L matemat_power-rescue:R-matemat_power-rescue R105
 U 1 1 50FB1B29
 P 5600 4950
@@
 $EndComp
 $Comp
-L matemat_power-rescue:C C101
+L matemat_power-rescue:C-matemat_power-rescue C101
 U 1 1 50FB1C81
 P 5250 4200
@@
 $EndComp
 $Comp
-L matemat_power-rescue:R R102
+L matemat_power-rescue:R-matemat_power-rescue R102
 U 1 1 50FB1CF2
 P 4950 4650
@@
 $EndComp
 $Comp
-L matemat_power-rescue:TRIAC_IEC T101
+L matemat_power-rescue:TRIAC_IEC-matemat_power-rescue T101
 U 1 1 50FB18FA
 P 5950 4550
@@
 $EndComp
 $Comp
-L matemat_power-rescue:GNDPWR #PWR01
+L matemat_power-rescue:GNDPWR-matemat_power-rescue #PWR01
 U 1 1 50FB1E40
 P 5250 4450
@@
 	5250 4450 5250 4400
 $Comp
-L matemat_power-rescue:GNDPWR #PWR02
+L matemat_power-rescue:GNDPWR-matemat_power-rescue #PWR02
 U 1 1 50FB1EFA
 P 5950 5250
@@
 	5950 5250 5950 4750
 $Comp
-L matemat_power-rescue:GNDPWR #PWR03
+L matemat_power-rescue:GNDPWR-matemat_power-rescue #PWR03
 U 1 1 50FB1F9D
 P 5600 5250
@@
 	5600 5250 5600 5200
 $Comp
-L matemat_power-rescue:GNDPWR #PWR04
+L matemat_power-rescue:GNDPWR-matemat_power-rescue #PWR04
 U 1 1 50FB1FD5
 P 6450 5250
@@
 	6450 4950 6450 5250
 $Comp
-L matemat_power-rescue:C C102
+L matemat_power-rescue:C-matemat_power-rescue C102
 U 1 1 50FB21D6
 P 6450 4750
@@
 $EndComp
 $Comp
-L matemat_power-rescue:CONN_2 J101
+L matemat_power-rescue:CONN_2-matemat_power-rescue J101
 U 1 1 50FB21F2
 P 6300 3350
@@
 $EndComp
 $Comp
-L matemat_power-rescue:HT #PWR05
+L matemat_power-rescue:HT-matemat_power-rescue #PWR05
 U 1 1 50FB22BF
 P 5950 2950
@@
 	3850 4850 3850 4650
 $Comp
-L matemat_power-rescue:GND #PWR06
+L matemat_power-rescue:GND-matemat_power-rescue #PWR06
 U 1 1 50FB2A82
 P 3850 4850
@@
 $EndComp
 $Comp
-L matemat_power-rescue:C C103
+L matemat_power-rescue:C-matemat_power-rescue C103
 U 1 1 50FB266D
 P 6900 4750

Commit message: Cleaned up schematics and removed obsolete parts
Parts:
- C101: footprint C2 -> Capacitor_THT:C_Rect_L7.0mm_W2.5mm_P5.00mm; symbol matemat_power-rescue:C-matemat_power-rescue -> Device:C
- C102: footprint cnp_18x5mm -> Capacitor_THT:C_Rect_L18.0mm_W5.0mm_P15.00mm_FKS3_FKP3; symbol matemat_power-rescue:C-matemat_power-rescue -> Device:C
- C103: footprint cnp_13x4mm -> Capacitor_THT:C_Rect_L13.0mm_W4.0mm_P10.00mm_FKS3_FKP3_MKS4; symbol matemat_power-rescue:C-matemat_power-rescue -> Device:C
- J101: footprint Bornier_B2_Wago -> TerminalBlock_WAGO:TerminalBlock_WAGO_236-102_1x02_P5.00mm_45Degree; symbol matemat_power-rescue:CONN_2-matemat_power-rescue -> Connector_Generic:Conn_01x02
- R101, R105: footprint SM0805 -> Resistor_SMD:R_0805_2012Metric_Pad1.20x1.40mm_HandSolder; symbol matemat_power-rescue:R-matemat_power-rescue -> Device:R
- R102, R103, R104: footprint through_R -> Resistor_THT:R_Axial_DIN0309_L9.0mm_D3.2mm_P12.70mm_Horizontal; symbol matemat_power-rescue:R-matemat_power-rescue -> Device:R
- T101: footprint _sto-TO220V -> Package_TO_SOT_THT:TO-220-3_Vertical; symbol matemat_power-rescue:TRIAC_IEC-matemat_power-rescue -> Triac_Thyristor:BT136-500
- U101: footprint TOpto_6 -> Package_DIP:DIP-6_W7.62mm_LongPads; symbol matemat_power-rescue:MOC3022M-matemat_power-rescue -> Relay_SolidState:MOC3022M
Connections:
- net GNDPWR renamed NEUT
- net HT renamed LINE

Commit message: Updated PCB layout
Parts:
- J101: footprint TerminalBlock_WAGO:TerminalBlock_WAGO_236-102_1x02_P5.00mm_45Degree -> TerminalBlock_WAGO:TerminalBlock_WAGO_236-402_1x02_P5.00mm_45Degree
Changed lines of the file:
@@
 F 0 "J101" H 6500 3450 50  0000 C CNN
 F 1 "Output" V 6350 3350 40  0000 C CNN
-F 2 "TerminalBlock_WAGO:TerminalBlock_WAGO_236-102_1x02_P5.00mm_45Degree" H 6300 3350 60  0001 C CNN
+F 2 "TerminalBlock_WAGO:TerminalBlock_WAGO_236-402_1x02_P5.00mm_45Degree" H 6300 3350 60  0001 C CNN
 F 3 "" H 6300 3350 60  0001 C CNN
 F 4 "FAR 1283527" H 6300 3350 60  0001 C CNN "Reference"
