File: power/triac_channel_6.sch (KiCad schematic (older format))
At the start: 11 parts, among them J601 Output, T601 BT136, U601 MOC3022M

Commit message: Updated power board for KiCAD 5
Parts:
- C601, C602, C603: symbol C -> matemat_power-rescue:C
- J601: symbol CONN_2 -> matemat_power-rescue:CONN_2
- R601, R602, R603, R604, R605: symbol R -> matemat_power-rescue:R
- T601: symbol TRIAC_IEC -> matemat_power-rescue:TRIAC_IEC
- U601: symbol MOC3022M -> matemat_power-rescue:MOC3022M
Changed lines of the file:
@@
-EESchema Schematic File Version 2
-LIBS:power
-LIBS:device
-LIBS:transistors
-LIBS:conn
-LIBS:linear
-LIBS:regul
-LIBS:74xx
-LIBS:cmos4000
-LIBS:adc-dac
-LIBS:memory
-LIBS:xilinx
-LIBS:special
-LIBS:microcontrollers
-LIBS:dsp
-LIBS:microchip
-LIBS:analog_switches
-LIBS:motorola
-LIBS:texas
-LIBS:intel
-LIBS:audio
-LIBS:interface
-LIBS:digital-audio
-LIBS:philips
-LIBS:display
-LIBS:cypress
-LIBS:siliconi
-LIBS:opto
-LIBS:atmel
-LIBS:contrib
-LIBS:valves
-LIBS:sto
-LIBS:sto2
-LIBS:40xx
-LIBS:uln-udn
-LIBS:optocoupler
-LIBS:diode-1_corr
+EESchema Schematic File Version 4
 LIBS:matemat_power-cache
-EELAYER 27 0
+EELAYER 26 0
 EELAYER END
 $Descr A4 11693 8268
@@
 $EndDescr
 $Comp
-L MOC3022M U601
+L matemat_power-rescue:MOC3022M U601
 U 1 1 50FB1912
 P 4200 4550
@@
 $EndComp
 $Comp
-L R R601
+L matemat_power-rescue:R R601
 U 1 1 50FB1948
 P 3850 4100
@@
 $EndComp
 $Comp
-L R R603
+L matemat_power-rescue:R R603
 U 1 1 50FB1B13
 P 5600 3850
@@
 $EndComp
 $Comp
-L R R604
+L matemat_power-rescue:R R604
 U 1 1 50FB1B1E
 P 6450 4200
@@
 $EndComp
 $Comp
-L R R605
+L matemat_power-rescue:R R605
 U 1 1 50FB1B29
 P 5600 4950
@@
 $EndComp
 $Comp
-L C C601
+L matemat_power-rescue:C C601
 U 1 1 50FB1C81
 P 5250 4200
@@
 $EndComp
 $Comp
-L R R602
+L matemat_power-rescue:R R602
 U 1 1 50FB1CF2
 P 4950 4650
@@
 $EndComp
 $Comp
-L TRIAC_IEC T601
+L matemat_power-rescue:TRIAC_IEC T601
 U 1 1 50FB18FA
 P 5950 4550
@@
 $EndComp
 $Comp
-L GNDPWR #PWR01
+L matemat_power-rescue:GNDPWR #PWR01
 U 1 1 50FB1E40
 P 5250 4450
@@
 	5250 4450 5250 4400
 $Comp
-L GNDPWR #PWR02
+L matemat_power-rescue:GNDPWR #PWR02
 U 1 1 50FB1EFA
 P 5950 5250
@@
 	5950 5250 5950 4750
 $Comp
-L GNDPWR #PWR03
+L matemat_power-rescue:GNDPWR #PWR03
 U 1 1 50FB1F9D
 P 5600 5250
@@
 	5600 5250 5600 5200
 $Comp
-L GNDPWR #PWR04
+L matemat_power-rescue:GNDPWR #PWR04
 U 1 1 50FB1FD5
 P 6450 5250
@@
 	6450 4950 6450 5250
 $Comp
-L C C602
+L matemat_power-rescue:C C602
 U 1 1 50FB21D6
 P 6450 4750
@@
 $EndComp
 $Comp
-L CONN_2 J601
+L matemat_power-rescue:CONN_2 J601
 U 1 1 50FB21F2
 P 6300 3350
@@
 $EndComp
 $Comp
-L HT #PWR05
+L matemat_power-rescue:HT #PWR05
 U 1 1 50FB22BF
 P 5950 2950
@@
 	3850 4850 3850 4650
 $Comp
-L GND #PWR06
+L matemat_power-rescue:GND #PWR06
 U 1 1 50FB2A82
 P 3850 4850
@@
 $EndComp
 $Comp
-L C C603
+L matemat_power-rescue:C C603
 U 1 1 50FB266D
 P 6900 4750

Commit message: Recreated rescue library
Parts:
- C601, C602, C603: symbol matemat_power-rescue:C -> matemat_power-rescue:C-matemat_power-rescue
- J601: symbol matemat_power-rescue:CONN_2 -> matemat_power-rescue:CONN_2-matemat_power-rescue
- R601, R602, R603, R604, R605: symbol matemat_power-rescue:R -> matemat_power-rescue:R-matemat_power-rescue
- T601: symbol matemat_power-rescue:TRIAC_IEC -> matemat_power-rescue:TRIAC_IEC-matemat_power-rescue
- U601: symbol matemat_power-rescue:MOC3022M -> matemat_power-rescue:MOC3022M-matemat_power-rescue
Changed lines of the file:
@@
 EESchema Schematic File Version 4
-LIBS:matemat_power-cache
-EELAYER 26 0
+EELAYER 30 0
 EELAYER END
 $Descr A4 11693 8268
@@
 $EndDescr
 $Comp
-L matemat_power-rescue:MOC3022M U601
+L matemat_power-rescue:MOC3022M-matemat_power-rescue U601
 U 1 1 50FB1912
 P 4200 4550
@@
 $EndComp
 $Comp
-L matemat_power-rescue:R R601
+L matemat_power-rescue:R-matemat_power-rescue R601
 U 1 1 50FB1948
 P 3850 4100
@@
 $EndComp
 $Comp
-L matemat_power-rescue:R R603
+L matemat_power-rescue:R-matemat_power-rescue R603
 U 1 1 50FB1B13
 P 5600 3850
@@
 $EndComp
 $Comp
-L matemat_power-rescue:R R604
+L matemat_power-rescue:R-matemat_power-rescue R604
 U 1 1 50FB1B1E
 P 6450 4200
@@
 $EndComp
 $Comp
-L matemat_power-rescue:R R605
+L matemat_power-rescue:R-matemat_power-rescue R605
 U 1 1 50FB1B29
 P 5600 4950
@@
 $EndComp
 $Comp
-L matemat_power-rescue:C C601
+L matemat_power-rescue:C-matemat_power-rescue C601
 U 1 1 50FB1C81
 P 5250 4200
@@
 $EndComp
 $Comp
-L matemat_power-rescue:R R602
+L matemat_power-rescue:R-matemat_power-rescue R602
 U 1 1 50FB1CF2
 P 4950 4650
@@
 $EndComp
 $Comp
-L matemat_power-rescue:TRIAC_IEC T601
+L matemat_power-rescue:TRIAC_IEC-matemat_power-rescue T601
 U 1 1 50FB18FA
 P 5950 4550
@@
 $EndComp
 $Comp
-L matemat_power-rescue:GNDPWR #PWR01
+L matemat_power-rescue:GNDPWR-matemat_power-rescue #PWR01
 U 1 1 50FB1E40
 P 5250 4450
@@
 	5250 4450 5250 4400
 $Comp
-L matemat_power-rescue:GNDPWR #PWR02
+L matemat_power-rescue:GNDPWR-matemat_power-rescue #PWR02
 U 1 1 50FB1EFA
 P 5950 5250
@@
 	5950 5250 5950 4750
 $Comp
-L matemat_power-rescue:GNDPWR #PWR03
+L matemat_power-rescue:GNDPWR-matemat_power-rescue #PWR03
 U 1 1 50FB1F9D
 P 5600 5250
@@
 	5600 5250 5600 5200
 $Comp
-L matemat_power-rescue:GNDPWR #PWR04
+L matemat_power-rescue:GNDPWR-matemat_power-rescue #PWR04
 U 1 1 50FB1FD5
 P 6450 5250
@@
 	6450 4950 6450 5250
 $Comp
-L matemat_power-rescue:C C602
+L matemat_power-rescue:C-matemat_power-rescue C602
 U 1 1 50FB21D6
 P 6450 4750
@@
 $EndComp
 $Comp
-L matemat_power-rescue:CONN_2 J601
+L matemat_power-rescue:CONN_2-matemat_power-rescue J601
 U 1 1 50FB21F2
 P 6300 3350
@@
 $EndComp
 $Comp
-L matemat_power-rescue:HT #PWR05
+L matemat_power-rescue:HT-matemat_power-rescue #PWR05
 U 1 1 50FB22BF
 P 5950 2950
@@
 	3850 4850 3850 4650
 $Comp
-L matemat_power-rescue:GND #PWR06
+L matemat_power-rescue:GND-matemat_power-rescue #PWR06
 U 1 1 50FB2A82
 P 3850 4850
@@
 $EndComp
 $Comp
-L matemat_power-rescue:C C603
+L matemat_power-rescue:C-matemat_power-rescue C603
 U 1 1 50FB266D
 P 6900 4750

Commit message: Cleaned up schematics and removed obsolete parts
Parts:
- C601: footprint C2 -> Capacitor_THT:C_Rect_L7.0mm_W2.5mm_P5.00mm; symbol matemat_power-rescue:C-matemat_power-rescue -> Device:C
- C602: footprint cnp_18x5mm -> Capacitor_THT:C_Rect_L18.0mm_W5.0mm_P15.00mm_FKS3_FKP3; symbol matemat_power-rescue:C-matemat_power-rescue -> Device:C
- C603: footprint cnp_13x4mm -> Capacitor_THT:C_Rect_L13.0mm_W4.0mm_P10.00mm_FKS3_FKP3_MKS4; symbol matemat_power-rescue:C-matemat_power-rescue -> Device:C
- J601: footprint Bornier_B2_Wago -> TerminalBlock_WAGO:TerminalBlock_WAGO_236-102_1x02_P5.00mm_45Degree; symbol matemat_power-rescue:CONN_2-matemat_power-rescue -> Connector_Generic:Conn_01x02
- R601, R605: footprint SM0805 -> Resistor_SMD:R_0805_2012Metric_Pad1.20x1.40mm_HandSolder; symbol matemat_power-rescue:R-matemat_power-rescue -> Device:R
- R602, R603, R604: footprint through_R -> Resistor_THT:R_Axial_DIN0309_L9.0mm_D3.2mm_P12.70mm_Horizontal; symbol matemat_power-rescue:R-matemat_power-rescue -> Device:R
- T601: footprint _sto-TO220V -> Package_TO_SOT_THT:TO-220-3_Vertical; symbol matemat_power-rescue:TRIAC_IEC-matemat_power-rescue -> Triac_Thyristor:BT136-500
- U601: footprint TOpto_6 -> Package_DIP:DIP-4_W7.62mm_LongPads; symbol matemat_power-rescue:MOC3022M-matemat_power-rescue -> Relay_SolidState:MOC3022M
Connections:
- net GNDPWR renamed NEUT
- net HT renamed LINE
Changed lines of the file:
@@
 $Descr A4 11693 8268
 encoding utf-8
-Sheet 1 11
+Sheet 8 11
 Title ""
 Date "19 jan 2013"
@@
 $EndDescr
 $Comp
-L matemat_power-rescue:MOC3022M-matemat_power-rescue U601
+L Relay_SolidState:MOC3022M U601
 U 1 1 50FB1912
 P 4200 4550
 F 0 "U601" H 3986 4729 40  0000 C CNN
 F 1 "MOC3022M" H 4300 4365 40  0000 C CNN
-F 2 "TOpto_6" H 4036 4375 29  0000 C CNN
-F 3 "" H 4200 4550 60  0001 C CNN
+F 2 "Package_DIP:DIP-4_W7.62mm_LongPads" H 4036 4375 29  0001 C CNN
+F 3 "https://www.onsemi.com/pub/Collateral/MOC3023M-D.PDF" H 4200 4550 60  0001 C CNN
 	1    4200 4550
 	1    0    0    -1
 $EndComp
 $Comp
-L matemat_power-rescue:R-matemat_power-rescue R601
+L Device:R R601
 U 1 1 50FB1948
 P 3850 4100
 F 0 "R601" V 3950 4100 50  0000 C CNN
 F 1 "1k" V 3850 4100 50  0000 C CNN
-F 2 "SM0805" H 3850 4100 60  0001 C CNN
+F 2 "Resistor_SMD:R_0805_2012Metric_Pad1.20x1.40mm_HandSolder" H 3850 4100 60  0001 C CNN
 F 3 "" H 3850 4100 60  0001 C CNN
 	1    3850 4100
@@
 $EndComp
 $Comp
-L matemat_power-rescue:R-matemat_power-rescue R603
+L Device:R R603
 U 1 1 50FB1B13
 P 5600 3850
 F 0 "R603" V 5500 3850 50  0000 C CNN
 F 1 "470" V 5600 3850 50  0000 C CNN
-F 2 "through_R" H 5600 3850 60  0001 C CNN
+F 2 "Resistor_THT:R_Axial_DIN0309_L9.0mm_D3.2mm_P12.70mm_Horizontal" H 5600 3850 60  0001 C CNN
 F 3 "" H 5600 3850 60  0001 C CNN
 	1    5600 3850
@@
 $EndComp
 $Comp
-L matemat_power-rescue:R-matemat_power-rescue R604
+L Device:R R604
 U 1 1 50FB1B1E
 P 6450 4200
 F 0 "R604" V 6350 4200 50  0000 C CNN
 F 1 "100" V 6450 4200 50  0000 C CNN
-F 2 "through_R" H 6450 4200 60  0001 C CNN
+F 2 "Resistor_THT:R_Axial_DIN0309_L9.0mm_D3.2mm_P12.70mm_Horizontal" H 6450 4200 60  0001 C CNN
 F 3 "" H 6450 4200 60  0001 C CNN
 	1    6450 4200
@@
 $EndComp
 $Comp
-L matemat_power-rescue:R-matemat_power-rescue R605
+L Device:R R605
 U 1 1 50FB1B29
 P 5600 4950
 F 0 "R605" V 5500 4950 50  0000 C CNN
 F 1 "100" V 5600 4950 50  0000 C CNN
-F 2 "SM0805" H 5600 4950 60  0001 C CNN
+F 2 "Resistor_SMD:R_0805_2012Metric_Pad1.20x1.40mm_HandSolder" H 5600 4950 60  0001 C CNN
 F 3 "" H 5600 4950 60  0001 C CNN
 	1    5600 4950
@@
 $EndComp
 $Comp
-L matemat_power-rescue:C-matemat_power-rescue C601
+L Device:C C601
 U 1 1 50FB1C81
 P 5250 4200
 F 0 "C601" H 4950 4300 50  0000 L CNN
 F 1 "10n" H 4950 4200 50  0000 L CNN
-F 2 "C2" V 5100 3950 60  0001 C CNN
+F 2 "Capacitor_THT:C_Rect_L7.0mm_W2.5mm_P5.00mm" V 5100 3950 60  0001 C CNN
 F 3 "" H 5250 4200 60  0001 C CNN
 	1    5250 4200
@@
 $EndComp
 $Comp
-L matemat_power-rescue:R-matemat_power-rescue R602
+L Device:R R602
 U 1 1 50FB1CF2
 P 4950 4650
 F 0 "R602" V 4850 4650 50  0000 C CNN
 F 1 "100" V 4950 4650 50  0000 C CNN
-F 2 "through_R" H 4950 4650 60  0001 C CNN
+F 2 "Resistor_THT:R_Axial_DIN0309_L9.0mm_D3.2mm_P12.70mm_Horizontal" H 4950 4650 60  0001 C CNN
 F 3 "" H 4950 4650 60  0001 C CNN
 	1    4950 4650
@@
 $EndComp
 $Comp
-L matemat_power-rescue:TRIAC_IEC-matemat_power-rescue T601
+L Triac_Thyristor:BT136-500 T601
 U 1 1 50FB18FA
 P 5950 4550
 F 0 "T601" V 5900 4750 40  0000 C CNN
 F 1 "BT136" V 6000 4750 40  0000 C CNN
-F 2 "_sto-TO220V" H 5950 4550 60  0001 C CNN
-F 3 "" H 5950 4550 60  0001 C CNN
+F 2 "Package_TO_SOT_THT:TO-220-3_Vertical" H 5950 4550 60  0001 C CNN
+F 3 "http://www.micropik.com/PDF/BT136-600.pdf" H 5950 4550 60  0001 C CNN
 	1    5950 4550
-	0    1    1    0
-$EndComp
-$Comp
-L matemat_power-rescue:GNDPWR-matemat_power-rescue #PWR01
-U 1 1 50FB1E40
-P 5250 4450
-F 0 "#PWR01" H 5250 4500 40  0001 C CNN
-F 1 "GNDPWR" H 5250 4370 40  0000 C CNN
-F 2 "" H 5250 4450 60  0001 C CNN
-F 3 "" H 5250 4450 60  0001 C CNN
-	1    5250 4450
-	1    0    0    -1
-$EndComp
-Wire Wire Line
-	5250 4450 5250 4400
-$Comp
-L matemat_power-rescue:GNDPWR-matemat_power-rescue #PWR02
-U 1 1 50FB1EFA
-P 5950 5250
-F 0 "#PWR02" H 5950 5300 40  0001 C CNN
-F 1 "GNDPWR" H 5950 5170 40  0000 C CNN
-F 2 "" H 5950 5250 60  0001 C CNN
-F 3 "" H 5950 5250 60  0001 C CNN
-	1    5950 5250
-	1    0    0    -1
-$EndComp
-Wire Wire Line
-	5950 5250 5950 4750
-$Comp
-L matemat_power-rescue:GNDPWR-matemat_power-rescue #PWR03
-U 1 1 50FB1F9D
-P 5600 5250
-F 0 "#PWR03" H 5600 5300 40  0001 C CNN
-F 1 "GNDPWR" H 5600 5170 40  0000 C CNN
-F 2 "" H 5600 5250 60  0001 C CNN
-F 3 "" H 5600 5250 60  0001 C CNN
-	1    5600 5250
-	1    0    0    -1
-$EndComp
-Wire Wire Line
-	5600 5250 5600 5200
-$Comp
-L matemat_power-rescue:GNDPWR-matemat_power-rescue #PWR04
-U 1 1 50FB1FD5
-P 6450 5250
-F 0 "#PWR04" H 6450 5300 40  0001 C CNN
-F 1 "GNDPWR" H 6450 5170 40  0000 C CNN
-F 2 "" H 6450 5250 60  0001 C CNN
-F 3 "" H 6450 5250 60  0001 C CNN
-	1    6450 5250
-	1    0    0    -1
-$EndComp
-Wire Wire Line
-	6450 4950 6450 5250
-$Comp
-L matemat_power-rescue:C-matemat_power-rescue C602
+	1    0    0    -1
+$EndComp
+$Comp
+L Device:C C602
 U 1 1 50FB21D6
 P 6450 4750
 F 0 "C602" H 6150 4850 50  0000 L CNN
 F 1 "220n" H 6150 4750 50  0000 L CNN
-F 2 "cnp_18x5mm" V 6300 4500 60  0001 C CNN
+F 2 "Capacitor_THT:C_Rect_L18.0mm_W5.0mm_P15.00mm_FKS3_FKP3" V 6300 4500 60  0001 C CNN
 F 3 "" H 6450 4750 60  0001 C CNN
 	1    6450 4750
@@
 $EndComp
 $Comp
-L matemat_power-rescue:CONN_2-matemat_power-rescue J601
+L Connector_Generic:Conn_01x02 J601
 U 1 1 50FB21F2
 P 6300 3350
 F 0 "J601" H 6500 3450 50  0000 C CNN
 F 1 "Output" V 6350 3350 40  0000 C CNN
-F 2 "Bornier_B2_Wago" H 6300 3350 60  0001 C CNN
+F 2 "TerminalBlock_WAGO:TerminalBlock_WAGO_236-102_1x02_P5.00mm_45Degree" H 6300 3350 60  0001 C CNN
 F 3 "" H 6300 3350 60  0001 C CNN
 F 4 "FAR 1283527" H 6300 3350 60  0001 C CNN "Reference"
@@
 	1    0    0    -1
 $EndComp
-$Comp
-L matemat_power-rescue:HT-matemat_power-rescue #PWR05
-U 1 1 50FB22BF
-P 5950 2950
-F 0 "#PWR05" H 5950 3070 20  0001 C CNN
-F 1 "HT" H 5950 3040 30  0000 C CNN
-F 2 "" H 5950 2950 60  0001 C CNN
-F 3 "" H 5950 2950 60  0001 C CNN
-	1    5950 2950
-	1    0    0    -1
-$EndComp
-Wire Wire Line
-	5950 2950 5950 3250
-Wire Wire Line
-	4550 3850 5350 3850
-Wire Wire Line
-	5250 4000 5250 3850
+Wire Wire Line
+	4550 3850 5250 3850
 Connection ~ 5250 3850
 Wire Wire Line
-	5950 3450 5950 4350
-Wire Wire Line
-	6450 4550 6450 4450
+	5950 3450 5950 3850
 Wire Wire Line
 	4550 4450 4550 3850
-Wire Wire Line
-	6450 3850 6450 3950
 Connection ~ 5950 3850
-Wire Wire Line
-	5850 3850 6450 3850
-Wire Wire Line
-	5600 4700 5600 4650
 Connection ~ 5600 4650
 Text HLabel 3400 3700 0    60   Input ~ 0
@@
 	3850 4850 3850 4650
 $Comp
-L matemat_power-rescue:GND-matemat_power-rescue #PWR06
-U 1 1 50FB2A82
-P 3850 4850
-F 0 "#PWR06" H 3850 4850 30  0001 C CNN
-F 1 "GND" H 3850 4780 30  0001 C CNN
-F 2 "" H 3850 4850 60  0001 C CNN
-F 3 "" H 3850 4850 60  0001 C CNN
-	1    3850 4850
-	1    0    0    -1
-$EndComp
-$Comp
-L matemat_power-rescue:C-matemat_power-rescue C603
+L Device:C C603
 U 1 1 50FB266D
 P 6900 4750
 F 0 "C603" H 6600 4850 50  0000 L CNN
 F 1 "DNP" H 6600 4750 50  0000 L CNN
-F 2 "cnp_13x4mm" V 6750 4500 60  0001 C CNN
+F 2 "Capacitor_THT:C_Rect_L13.0mm_W4.0mm_P10.00mm_FKS3_FKP3_MKS4" V 6750 4500 60  0001 C CNN
 F 3 "" H 6900 4750 60  0001 C CNN
 	1    6900 4750
@@
 Wire Wire Line
 	6450 5000 6900 5000
-Wire Wire Line
-	6900 5000 6900 4950
 Connection ~ 6450 5000
-Wire Wire Line
-	6900 4550 6900 4500
 Wire Wire Line
 	6900 4500 6450 4500
 Connection ~ 6450 4500
 Wire Wire Line
-	4550 4650 4700 4650
-Wire Wire Line
-	5200 4650 5800 4650
-Wire Wire Line
 	3400 3700 3850 3700
 Wire Wire Line
-	3850 3700 3850 3850
-Wire Wire Line
-	3850 4350 3850 4450
+	5950 3850 6450 3850
+Wire Wire Line
+	5600 4650 5800 4650
+Wire Wire Line
+	6450 5000 6450 5250
+$Comp
+L power:LINE #PWR?
+U 1 1 604147DF
+P 5950 2950
+F 0 "#PWR?" H 5950 2800 50  0001 C CNN
+F 1 "LINE" H 5965 3123 50  0000 C CNN
+F 2 "" H 5950 2950 50  0001 C CNN
+F 3 "" H 5950 2950 50  0001 C CNN
+	1    5950 2950
+	1    0    0    -1
+$EndComp
+$Comp
+L power:NEUT #PWR?
+U 1 1 604150DD
+P 5250 4350
+F 0 "#PWR?" H 5250 4200 50  0001 C CNN
+F 1 "NEUT" H 5265 4523 50  0000 C CNN
+F 2 "" H 5250 4350 50  0001 C CNN
+F 3 "" H 5250 4350 50  0001 C CNN
+	1    5250 4350
+	-1   0    0    1
+$EndComp
+$Comp
+L power:NEUT #PWR?
+U 1 1 60415798
+P 5600 5250
+F 0 "#PWR?" H 5600 5100 50  0001 C CNN
+F 1 "NEUT" H 5615 5423 50  0000 C CNN
+F 2 "" H 5600 5250 50  0001 C CNN
+F 3 "" H 5600 5250 50  0001 C CNN
+	1    5600 5250
+	-1   0    0    1
+$EndComp
+$Comp
+L power:NEUT #PWR?
+U 1 1 60415ABF
+P 5950 5250
+F 0 "#PWR?" H 5950 5100 50  0001 C CNN
+F 1 "NEUT" H 5965 5423 50  0000 C CNN
+F 2 "" H 5950 5250 50  0001 C CNN
+F 3 "" H 5950 5250 50  0001 C CNN
+	1    5950 5250
+	-1   0    0    1
+$EndComp
+$Comp
+L power:NEUT #PWR?
+U 1 1 60415CED
+P 6450 5250
+F 0 "#PWR?" H 6450 5100 50  0001 C CNN
+F 1 "NEUT" H 6465 5423 50  0000 C CNN
+F 2 "" H 6450 5250 50  0001 C CNN
+F 3 "" H 6450 5250 50  0001 C CNN
+	1    6450 5250
+	-1   0    0    1
+$EndComp
+$Comp
+L power:GND #PWR?
+U 1 1 604162EA
+P 3850 4850
+F 0 "#PWR?" H 3850 4600 50  0001 C CNN
+F 1 "GND" H 3855 4677 50  0000 C CNN
+F 2 "" H 3850 4850 50  0001 C CNN
+F 3 "" H 3850 4850 50  0001 C CNN
+	1    3850 4850
+	1    0    0    -1
+$EndComp
+Wire Wire Line
+	6100 3350 5950 3350
+Wire Wire Line
+	5950 2950 5950 3350
+Wire Wire Line
+	6100 3450 5950 3450
+Wire Wire Line
+	3850 3700 3850 3950
+Wire Wire Line
+	3850 4250 3850 4450
+Wire Wire Line
+	3900 4450 3850 4450
+Wire Wire Line
+	3850 4650 3900 4650
+Wire Wire Line
+	4500 4450 4550 4450
+Wire Wire Line
+	4500 4650 4800 4650
+Wire Wire Line
+	5100 4650 5600 4650
+Wire Wire Line
+	5250 3850 5450 3850
+Wire Wire Line
+	5750 3850 5950 3850
+Wire Wire Line
+	5600 4650 5600 4800
+Wire Wire Line
+	5600 5100 5600 5250
+Wire Wire Line
+	5950 4700 5950 5250
+Wire Wire Line
+	6450 4350 6450 4500
+Wire Wire Line
+	6450 3850 6450 4050
+Wire Wire Line
+	6450 4500 6450 4600
+Wire Wire Line
+	6900 4500 6900 4600
+Wire Wire Line
+	6900 4900 6900 5000
+Wire Wire Line
+	6450 4900 6450 5000
+Wire Wire Line
+	5950 3850 5950 4400
+Wire Wire Line
+	5250 3850 5250 4050
 $EndSCHEMATC

Commit message: Updated PCB layout
Parts:
- J601: footprint TerminalBlock_WAGO:TerminalBlock_WAGO_236-102_1x02_P5.00mm_45Degree -> TerminalBlock_WAGO:TerminalBlock_WAGO_236-402_1x02_P5.00mm_45Degree
- U601: footprint Package_DIP:DIP-4_W7.62mm_LongPads -> Package_DIP:DIP-6_W7.62mm_LongPads
Changed lines of the file:
@@
 F 0 "U601" H 3986 4729 40  0000 C CNN
 F 1 "MOC3022M" H 4300 4365 40  0000 C CNN
-F 2 "Package_DIP:DIP-4_W7.62mm_LongPads" H 4036 4375 29  0001 C CNN
+F 2 "Package_DIP:DIP-6_W7.62mm_LongPads" H 4036 4375 29  0001 C CNN
 F 3 "https://www.onsemi.com/pub/Collateral/MOC3023M-D.PDF" H 4200 4550 60  0001 C CNN
 	1    4200 4550
@@
 F 0 "J601" H 6500 3450 50  0000 C CNN
 F 1 "Output" V 6350 3350 40  0000 C CNN
-F 2 "TerminalBlock_WAGO:TerminalBlock_WAGO_236-102_1x02_P5.00mm_45Degree" H 6300 3350 60  0001 C CNN
+F 2 "TerminalBlock_WAGO:TerminalBlock_WAGO_236-402_1x02_P5.00mm_45Degree" H 6300 3350 60  0001 C CNN
 F 3 "" H 6300 3350 60  0001 C CNN
 F 4 "FAR 1283527" H 6300 3350 60  0001 C CNN "Reference"
@@
 	6450 5000 6450 5250
 $Comp
-L power:LINE #PWR?
+L power:LINE #PWR0154
 U 1 1 604147DF
 P 5950 2950
-F 0 "#PWR?" H 5950 2800 50  0001 C CNN
+F 0 "#PWR0154" H 5950 2800 50  0001 C CNN
 F 1 "LINE" H 5965 3123 50  0000 C CNN
 F 2 "" H 5950 2950 50  0001 C CNN
@@
 $EndComp
 $Comp
-L power:NEUT #PWR?
+L power:NEUT #PWR0155
 U 1 1 604150DD
 P 5250 4350
-F 0 "#PWR?" H 5250 4200 50  0001 C CNN
+F 0 "#PWR0155" H 5250 4200 50  0001 C CNN
 F 1 "NEUT" H 5265 4523 50  0000 C CNN
 F 2 "" H 5250 4350 50  0001 C CNN
@@
 $EndComp
 $Comp
-L power:NEUT #PWR?
+L power:NEUT #PWR0156
 U 1 1 60415798
 P 5600 5250
-F 0 "#PWR?" H 5600 5100 50  0001 C CNN
+F 0 "#PWR0156" H 5600 5100 50  0001 C CNN
 F 1 "NEUT" H 5615 5423 50  0000 C CNN
 F 2 "" H 5600 5250 50  0001 C CNN
@@
 $EndComp
 $Comp
-L power:NEUT #PWR?
+L power:NEUT #PWR0157
 U 1 1 60415ABF
 P 5950 5250
-F 0 "#PWR?" H 5950 5100 50  0001 C CNN
+F 0 "#PWR0157" H 5950 5100 50  0001 C CNN
 F 1 "NEUT" H 5965 5423 50  0000 C CNN
 F 2 "" H 5950 5250 50  0001 C CNN
@@
 $EndComp
 $Comp
-L power:NEUT #PWR?
+L power:NEUT #PWR0158
 U 1 1 60415CED
 P 6450 5250
-F 0 "#PWR?" H 6450 5100 50  0001 C CNN
+F 0 "#PWR0158" H 6450 5100 50  0001 C CNN
 F 1 "NEUT" H 6465 5423 50  0000 C CNN
 F 2 "" H 6450 5250 50  0001 C CNN
@@
 $EndComp
 $Comp
-L power:GND #PWR?
+L power:GND #PWR0159
 U 1 1 604162EA
 P 3850 4850
-F 0 "#PWR?" H 3850 4600 50  0001 C CNN
+F 0 "#PWR0159" H 3850 4600 50  0001 C CNN
 F 1 "GND" H 3855 4677 50  0000 C CNN
 F 2 "" H 3850 4850 50  0001 C CNN
