File: power/triac_channel_8.sch (KiCad schematic (older format))
At the start: 11 parts, among them J801 Output, T801 BT136, U801 MOC3022M

Commit message: Updated power board for KiCAD 5
Parts:
- C801, C802, C803: symbol C -> matemat_power-rescue:C
- J801: symbol CONN_2 -> matemat_power-rescue:CONN_2
- R801, R802, R803, R804, R805: symbol R -> matemat_power-rescue:R
- T801: symbol TRIAC_IEC -> matemat_power-rescue:TRIAC_IEC
- U801: symbol MOC3022M -> matemat_power-rescue:MOC3022M
Changed lines of the file:
@@
-EESchema Schematic File Version 2
-LIBS:power
-LIBS:device
-LIBS:transistors
-LIBS:conn
-LIBS:linear
-LIBS:regul
-LIBS:74xx
-LIBS:cmos4000
-LIBS:adc-dac
-LIBS:memory
-LIBS:xilinx
-LIBS:special
-LIBS:microcontrollers
-LIBS:dsp
-LIBS:microchip
-LIBS:analog_switches
-LIBS:motorola
-LIBS:texas
-LIBS:intel
-LIBS:audio
-LIBS:interface
-LIBS:digital-audio
-LIBS:philips
-LIBS:display
-LIBS:cypress
-LIBS:siliconi
-LIBS:opto
-LIBS:atmel
-LIBS:contrib
-LIBS:valves
-LIBS:sto
-LIBS:sto2
-LIBS:40xx
-LIBS:uln-udn
-LIBS:optocoupler
-LIBS:diode-1_corr
+EESchema Schematic File Version 4
 LIBS:matemat_power-cache
-EELAYER 27 0
+EELAYER 26 0
 EELAYER END
 $Descr A4 11693 8268
@@
 $EndDescr
 $Comp
-L MOC3022M U801
+L matemat_power-rescue:MOC3022M U801
 U 1 1 50FB1912
 P 4200 4550
@@
 $EndComp
 $Comp
-L R R801
+L matemat_power-rescue:R R801
 U 1 1 50FB1948
 P 3850 4100
@@
 $EndComp
 $Comp
-L R R803
+L matemat_power-rescue:R R803
 U 1 1 50FB1B13
 P 5600 3850
@@
 $EndComp
 $Comp
-L R R804
+L matemat_power-rescue:R R804
 U 1 1 50FB1B1E
 P 6450 4200
@@
 $EndComp
 $Comp
-L R R805
+L matemat_power-rescue:R R805
 U 1 1 50FB1B29
 P 5600 4950
@@
 $EndComp
 $Comp
-L C C801
+L matemat_power-rescue:C C801
 U 1 1 50FB1C81
 P 5250 4200
@@
 $EndComp
 $Comp
-L R R802
+L matemat_power-rescue:R R802
 U 1 1 50FB1CF2
 P 4950 4650
@@
 $EndComp
 $Comp
-L TRIAC_IEC T801
+L matemat_power-rescue:TRIAC_IEC T801
 U 1 1 50FB18FA
 P 5950 4550
@@
 $EndComp
 $Comp
-L GNDPWR #PWR01
+L matemat_power-rescue:GNDPWR #PWR01
 U 1 1 50FB1E40
 P 5250 4450
@@
 	5250 4450 5250 4400
 $Comp
-L GNDPWR #PWR02
+L matemat_power-rescue:GNDPWR #PWR02
 U 1 1 50FB1EFA
 P 5950 5250
@@
 	5950 5250 5950 4750
 $Comp
-L GNDPWR #PWR03
+L matemat_power-rescue:GNDPWR #PWR03
 U 1 1 50FB1F9D
 P 5600 5250
@@
 	5600 5250 5600 5200
 $Comp
-L GNDPWR #PWR04
+L matemat_power-rescue:GNDPWR #PWR04
 U 1 1 50FB1FD5
 P 6450 5250
@@
 	6450 4950 6450 5250
 $Comp
-L C C802
+L matemat_power-rescue:C C802
 U 1 1 50FB21D6
 P 6450 4750
@@
 $EndComp
 $Comp
-L CONN_2 J801
+L matemat_power-rescue:CONN_2 J801
 U 1 1 50FB21F2
 P 6300 3350
@@
 $EndComp
 $Comp
-L HT #PWR05
+L matemat_power-rescue:HT #PWR05
 U 1 1 50FB22BF
 P 5950 2950
@@
 	3850 4850 3850 4650
 $Comp
-L GND #PWR06
+L matemat_power-rescue:GND #PWR06
 U 1 1 50FB2A82
 P 3850 4850
@@
 $EndComp
 $Comp
-L C C803
+L matemat_power-rescue:C C803
 U 1 1 50FB266D
 P 6900 4750

Commit message: Recreated rescue library
Parts:
- C801, C802, C803: symbol matemat_power-rescue:C -> matemat_power-rescue:C-matemat_power-rescue
- J801: symbol matemat_power-rescue:CONN_2 -> matemat_power-rescue:CONN_2-matemat_power-rescue
- R801, R802, R803, R804, R805: symbol matemat_power-rescue:R -> matemat_power-rescue:R-matemat_power-rescue
- T801: symbol matemat_power-rescue:TRIAC_IEC -> matemat_power-rescue:TRIAC_IEC-matemat_power-rescue
- U801: symbol matemat_power-rescue:MOC3022M -> matemat_power-rescue:MOC3022M-matemat_power-rescue
Changed lines of the file:
@@
 EESchema Schematic File Version 4
-LIBS:matemat_power-cache
-EELAYER 26 0
+EELAYER 30 0
 EELAYER END
 $Descr A4 11693 8268
@@
 $EndDescr
 $Comp
-L matemat_power-rescue:MOC3022M U801
+L matemat_power-rescue:MOC3022M-matemat_power-rescue U801
 U 1 1 50FB1912
 P 4200 4550
@@
 $EndComp
 $Comp
-L matemat_power-rescue:R R801
+L matemat_power-rescue:R-matemat_power-rescue R801
 U 1 1 50FB1948
 P 3850 4100
@@
 $EndComp
 $Comp
-L matemat_power-rescue:R R803
+L matemat_power-rescue:R-matemat_power-rescue R803
 U 1 1 50FB1B13
 P 5600 3850
@@
 $EndComp
 $Comp
-L matemat_power-rescue:R R804
+L matemat_power-rescue:R-matemat_power-rescue R804
 U 1 1 50FB1B1E
 P 6450 4200
@@
 $EndComp
 $Comp
-L matemat_power-rescue:R R805
+L matemat_power-rescue:R-matemat_power-rescue R805
 U 1 1 50FB1B29
 P 5600 4950
@@
 $EndComp
 $Comp
-L matemat_power-rescue:C C801
+L matemat_power-rescue:C-matemat_power-rescue C801
 U 1 1 50FB1C81
 P 5250 4200
@@
 $EndComp
 $Comp
-L matemat_power-rescue:R R802
+L matemat_power-rescue:R-matemat_power-rescue R802
 U 1 1 50FB1CF2
 P 4950 4650
@@
 $EndComp
 $Comp
-L matemat_power-rescue:TRIAC_IEC T801
+L matemat_power-rescue:TRIAC_IEC-matemat_power-rescue T801
 U 1 1 50FB18FA
 P 5950 4550
@@
 $EndComp
 $Comp
-L matemat_power-rescue:GNDPWR #PWR01
+L matemat_power-rescue:GNDPWR-matemat_power-rescue #PWR01
 U 1 1 50FB1E40
 P 5250 4450
@@
 	5250 4450 5250 4400
 $Comp
-L matemat_power-rescue:GNDPWR #PWR02
+L matemat_power-rescue:GNDPWR-matemat_power-rescue #PWR02
 U 1 1 50FB1EFA
 P 5950 5250
@@
 	5950 5250 5950 4750
 $Comp
-L matemat_power-rescue:GNDPWR #PWR03
+L matemat_power-rescue:GNDPWR-matemat_power-rescue #PWR03
 U 1 1 50FB1F9D
 P 5600 5250
@@
 	5600 5250 5600 5200
 $Comp
-L matemat_power-rescue:GNDPWR #PWR04
+L matemat_power-rescue:GNDPWR-matemat_power-rescue #PWR04
 U 1 1 50FB1FD5
 P 6450 5250
@@
 	6450 4950 6450 5250
 $Comp
-L matemat_power-rescue:C C802
+L matemat_power-rescue:C-matemat_power-rescue C802
 U 1 1 50FB21D6
 P 6450 4750
@@
 $EndComp
 $Comp
-L matemat_power-rescue:CONN_2 J801
+L matemat_power-rescue:CONN_2-matemat_power-rescue J801
 U 1 1 50FB21F2
 P 6300 3350
@@
 $EndComp
 $Comp
-L matemat_power-rescue:HT #PWR05
+L matemat_power-rescue:HT-matemat_power-rescue #PWR05
 U 1 1 50FB22BF
 P 5950 2950
@@
 	3850 4850 3850 4650
 $Comp
-L matemat_power-rescue:GND #PWR06
+L matemat_power-rescue:GND-matemat_power-rescue #PWR06
 U 1 1 50FB2A82
 P 3850 4850
@@
 $EndComp
 $Comp
-L matemat_power-rescue:C C803
+L matemat_power-rescue:C-matemat_power-rescue C803
 U 1 1 50FB266D
 P 6900 4750

Commit message: Cleaned up schematics and removed obsolete parts
Parts:
- C801: footprint C2 -> Capacitor_THT:C_Rect_L7.0mm_W2.5mm_P5.00mm; symbol matemat_power-rescue:C-matemat_power-rescue -> Device:C
- C802: footprint cnp_18x5mm -> Capacitor_THT:C_Rect_L18.0mm_W5.0mm_P15.00mm_FKS3_FKP3; symbol matemat_power-rescue:C-matemat_power-rescue -> Device:C
- C803: footprint cnp_13x4mm -> Capacitor_THT:C_Rect_L13.0mm_W4.0mm_P10.00mm_FKS3_FKP3_MKS4; symbol matemat_power-rescue:C-matemat_power-rescue -> Device:C
- J801: footprint Bornier_B2_Wago -> TerminalBlock_WAGO:TerminalBlock_WAGO_236-102_1x02_P5.00mm_45Degree; symbol matemat_power-rescue:CONN_2-matemat_power-rescue -> Connector_Generic:Conn_01x02
- R801, R805: footprint SM0805 -> Resistor_SMD:R_0805_2012Metric_Pad1.20x1.40mm_HandSolder; symbol matemat_power-rescue:R-matemat_power-rescue -> Device:R
- R802, R803, R804: footprint through_R -> Resistor_THT:R_Axial_DIN0309_L9.0mm_D3.2mm_P12.70mm_Horizontal; symbol matemat_power-rescue:R-matemat_power-rescue -> Device:R
- T801: footprint _sto-TO220V -> Package_TO_SOT_THT:TO-220-3_Vertical; symbol matemat_power-rescue:TRIAC_IEC-matemat_power-rescue -> Triac_Thyristor:BT136-500
- U801: footprint TOpto_6 -> Package_DIP:DIP-4_W7.62mm_LongPads; symbol matemat_power-rescue:MOC3022M-matemat_power-rescue -> Relay_SolidState:MOC3022M
Connections:
- net GNDPWR renamed NEUT
- net HT renamed LINE

Commit message: Updated PCB layout
Parts:
- J801: footprint TerminalBlock_WAGO:TerminalBlock_WAGO_236-102_1x02_P5.00mm_45Degree -> TerminalBlock_WAGO:TerminalBlock_WAGO_236-402_1x02_P5.00mm_45Degree
- U801: footprint Package_DIP:DIP-4_W7.62mm_LongPads -> Package_DIP:DIP-6_W7.62mm_LongPads
Changed lines of the file:
@@
 F 0 "U801" H 3986 4729 40  0000 C CNN
 F 1 "MOC3022M" H 4300 4365 40  0000 C CNN
-F 2 "Package_DIP:DIP-4_W7.62mm_LongPads" H 4036 4375 29  0001 C CNN
+F 2 "Package_DIP:DIP-6_W7.62mm_LongPads" H 4036 4375 29  0001 C CNN
 F 3 "https://www.onsemi.com/pub/Collateral/MOC3023M-D.PDF" H 4200 4550 60  0001 C CNN
 	1    4200 4550
@@
 F 0 "J801" H 6500 3450 50  0000 C CNN
 F 1 "Output" V 6350 3350 40  0000 C CNN
-F 2 "TerminalBlock_WAGO:TerminalBlock_WAGO_236-102_1x02_P5.00mm_45Degree" H 6300 3350 60  0001 C CNN
+F 2 "TerminalBlock_WAGO:TerminalBlock_WAGO_236-402_1x02_P5.00mm_45Degree" H 6300 3350 60  0001 C CNN
 F 3 "" H 6300 3350 60  0001 C CNN
 F 4 "FAR 1283527" H 6300 3350 60  0001 C CNN "Reference"
@@
 	6450 5000 6450 5250
 $Comp
-L power:LINE #PWR?
+L power:LINE #PWR0183
 U 1 1 60438FA7
 P 5950 2950
-F 0 "#PWR?" H 5950 2800 50  0001 C CNN
+F 0 "#PWR0183" H 5950 2800 50  0001 C CNN
 F 1 "LINE" H 5965 3123 50  0000 C CNN
 F 2 "" H 5950 2950 50  0001 C CNN
@@
 $EndComp
 $Comp
-L power:GND #PWR?
+L power:GND #PWR0184
 U 1 1 6043944B
 P 3850 4850
-F 0 "#PWR?" H 3850 4600 50  0001 C CNN
+F 0 "#PWR0184" H 3850 4600 50  0001 C CNN
 F 1 "GND" H 3855 4677 50  0000 C CNN
 F 2 "" H 3850 4850 50  0001 C CNN
@@
 $EndComp
 $Comp
-L power:NEUT #PWR?
+L power:NEUT #PWR0185
 U 1 1 6043977F
 P 5250 4400
-F 0 "#PWR?" H 5250 4250 50  0001 C CNN
+F 0 "#PWR0185" H 5250 4250 50  0001 C CNN
 F 1 "NEUT" H 5265 4573 50  0000 C CNN
 F 2 "" H 5250 4400 50  0001 C CNN
@@
 $EndComp
 $Comp
-L power:NEUT #PWR?
+L power:NEUT #PWR0186
 U 1 1 6043983F
 P 5600 5250
-F 0 "#PWR?" H 5600 5100 50  0001 C CNN
+F 0 "#PWR0186" H 5600 5100 50  0001 C CNN
 F 1 "NEUT" H 5615 5423 50  0000 C CNN
 F 2 "" H 5600 5250 50  0001 C CNN
@@
 $EndComp
 $Comp
-L power:NEUT #PWR?
+L power:NEUT #PWR0187
 U 1 1 60439B62
 P 5950 5250
-F 0 "#PWR?" H 5950 5100 50  0001 C CNN
+F 0 "#PWR0187" H 5950 5100 50  0001 C CNN
 F 1 "NEUT" H 5965 5423 50  0000 C CNN
 F 2 "" H 5950 5250 50  0001 C CNN
@@
 $EndComp
 $Comp
-L power:NEUT #PWR?
+L power:NEUT #PWR0188
 U 1 1 60439D76
 P 6450 5250
-F 0 "#PWR?" H 6450 5100 50  0001 C CNN
+F 0 "#PWR0188" H 6450 5100 50  0001 C CNN
 F 1 "NEUT" H 6465 5423 50  0000 C CNN
 F 2 "" H 6450 5250 50  0001 C CNN
