File: power/outputs.sch (KiCad schematic (older format))
At the start: 22 parts, among them IC1 4094D, IC2 4094D, IC3 ULN2803A, IC4 PC817, J11 CONN_8, J4 MAIN_BOARD_BUS, Q1 NPN_BCE

Commit message: Updated power board for KiCAD 5
Parts:
- C3, C4: symbol C -> matemat_power-rescue:C
- D10, D11, D6, D9: symbol DIODE -> matemat_power-rescue:DIODE
- D12: symbol BZX84CSMD -> matemat_power-rescue:BZX84CSMD
- IC1, IC2: symbol 4094D -> matemat_power-rescue:4094D
- IC3: symbol ULN2803A -> matemat_power-rescue:ULN2803A
- IC4: symbol PC817 -> matemat_power-rescue:PC817
- J11: symbol CONN_8 -> matemat_power-rescue:CONN_8
- J4: symbol BUS_I2C -> matemat:Bus_I2C
- JMP1, JMP2, R1, R2, R3, R4, R5, R6: symbol R -> matemat_power-rescue:R
- Q1: symbol NPN_BCE -> matemat_power-rescue:NPN_BCE
Connections:
- wire segments 118 -> 132
Changed lines of the file:
@@
-EESchema Schematic File Version 2
-LIBS:power
-LIBS:device
-LIBS:transistors
-LIBS:conn
-LIBS:linear
-LIBS:regul
-LIBS:74xx
-LIBS:cmos4000
-LIBS:adc-dac
-LIBS:memory
-LIBS:xilinx
-LIBS:special
-LIBS:microcontrollers
-LIBS:dsp
-LIBS:microchip
-LIBS:analog_switches
-LIBS:motorola
-LIBS:texas
-LIBS:intel
-LIBS:audio
-LIBS:interface
-LIBS:digital-audio
-LIBS:philips
-LIBS:display
-LIBS:cypress
-LIBS:siliconi
-LIBS:opto
-LIBS:atmel
-LIBS:contrib
-LIBS:valves
-LIBS:sto
-LIBS:sto2
-LIBS:40xx
-LIBS:uln-udn
-LIBS:optocoupler
-LIBS:diode-1_corr
+EESchema Schematic File Version 4
 LIBS:matemat_power-cache
-EELAYER 27 0
+EELAYER 26 0
 EELAYER END
 $Descr A4 11693 8268
@@
 $EndDescr
 $Comp
-L +12V #PWR11
+L matemat_power-rescue:+12V #PWR11
 U 1 1 50F5F502
 P 4550 6900
@@
 $EndComp
 $Comp
-L +5V #PWR10
+L matemat_power-rescue:+5V #PWR10
 U 1 1 50F5F508
 P 2850 6800
@@
 $EndComp
 $Comp
-L GND #PWR12
+L matemat_power-rescue:GND #PWR12
 U 1 1 50F5F50E
 P 4600 6800
@@
 $EndComp
 $Comp
-L BUS_I2C J4
+L matemat:Bus_I2C J4
 U 1 1 50F5F5BF
 P 3650 7150
+AR Path="/50F5F5BF" Ref="J4"  Part="1"
+AR Path="/50F5F19D/50F5F5BF" Ref="J4"  Part="1"
 F 0 "J4" H 3650 7600 70  0000 C CNN
 F 1 "MAIN_BOARD_BUS" H 3600 6650 70  0000 C CNN
@@
 $EndComp
 $Comp
-L 4094D IC1
+L matemat_power-rescue:4094D IC1
 U 1 1 50F5F7F4
 P 2600 5550
@@
 strobe
 $Comp
-L R JMP1
+L matemat_power-rescue:R JMP1
 U 1 1 50F5F6F8
 P 2550 7500
@@
 $EndComp
 $Comp
-L +5V #PWR9
+L matemat_power-rescue:+5V #PWR9
 U 1 1 50F5FA42
 P 2400 6250
@@
 $EndComp
 $Comp
-L R JMP2
+L matemat_power-rescue:R JMP2
 U 1 1 50F5FB5C
 P 2550 7650
@@
 $EndSheet
 $Comp
-L +5V #PWR5
+L matemat_power-rescue:+5V #PWR5
 U 1 1 50FF3F43
 P 1450 4950
@@
 $EndComp
 $Comp
-L 4094D IC1
+L matemat_power-rescue:4094D IC1
 U 2 1 5105769F
 P 1450 5350
@@
 $EndComp
 $Comp
-L C C3
+L matemat_power-rescue:C C3
 U 1 1 510583BD
 P 1000 5300
@@
 $EndComp
 $Comp
-L GND #PWR6
+L matemat_power-rescue:GND #PWR6
 U 1 1 5105853A
 P 1450 5750
@@
 $EndComp
 $Comp
-L 4094D IC2
+L matemat_power-rescue:4094D IC2
 U 1 1 510836A5
 P 6800 6350
@@
 $EndComp
 $Comp
-L ULN2803A IC3
+L matemat_power-rescue:ULN2803A IC3
 U 1 1 51086ED4
 P 8350 5150
@@
 $EndComp
 $Comp
-L +5V #PWR13
+L matemat_power-rescue:+5V #PWR13
 U 1 1 510872E7
 P 5800 6000
@@
 $EndComp
 $Comp
-L 4094D IC2
+L matemat_power-rescue:4094D IC2
 U 2 1 510872ED
 P 5800 6400
@@
 $EndComp
 $Comp
-L C C4
+L matemat_power-rescue:C C4
 U 1 1 510872F3
 P 5350 6350
@@
 $EndComp
 $Comp
-L GND #PWR14
+L matemat_power-rescue:GND #PWR14
 U 1 1 51087300
 P 5800 6800
@@
 strobe
 $Comp
-L +5V #PWR16
+L matemat_power-rescue:+5V #PWR16
 U 1 1 51088412
 P 6600 7050
@@
 Dout1_Din2
 $Comp
-L GND #PWR17
+L matemat_power-rescue:GND #PWR17
 U 1 1 510888ED
 P 7850 5800
@@
 $EndComp
 $Comp
-L CONN_8 J11
+L matemat_power-rescue:CONN_8 J11
 U 1 1 5108C0AA
 P 9600 5100
@@
 $EndComp
 $Comp
-L +12V #PWR20
+L matemat_power-rescue:+12V #PWR20
 U 1 1 5108D085
 P 9100 5800
@@
 $EndComp
 $Comp
-L R R1
+L matemat_power-rescue:R R1
 U 1 1 5108F808
 P 2250 7000
@@
 $EndComp
 $Comp
-L R R2
+L matemat_power-rescue:R R2
 U 1 1 5108FCDB
 P 2250 7100
@@
 $EndComp
 $Comp
-L +5V #PWR7
+L matemat_power-rescue:+5V #PWR7
 U 1 1 5108FE16
 P 1750 7000
@@
 $EndComp
 $Comp
-L +5V #PWR8
+L matemat_power-rescue:+5V #PWR8
 U 1 1 5108FE1C
 P 1750 7100
@@
 $EndComp
 $Comp
-L R R5
+L matemat_power-rescue:R R5
 U 1 1 51093461
 P 8150 3350
@@
 $EndComp
 $Comp
-L HT #PWR15
+L matemat_power-rescue:HT #PWR15
 U 1 1 51093496
 P 6250 2300
@@
 $EndComp
 $Comp
-L PC817 IC4
+L matemat_power-rescue:PC817 IC4
 U 1 1 510964E4
 P 8500 2950
@@
 $EndComp
 $Comp
-L R R6
+L matemat_power-rescue:R R6
 U 1 1 51096DB7
 P 8850 2350
@@
 $EndComp
 $Comp
-L DIODE D6
+L matemat_power-rescue:DIODE D6
 U 1 1 51097ED5
 P 6750 2600
@@
 $EndComp
 $Comp
-L DIODE D9
+L matemat_power-rescue:DIODE D9
 U 1 1 51097EDD
 P 6750 3200
@@
 $EndComp
 $Comp
-L DIODE D10
+L matemat_power-rescue:DIODE D10
 U 1 1 51097EE5
 P 7250 2600
@@
 $EndComp
 $Comp
-L DIODE D11
+L matemat_power-rescue:DIODE D11
 U 1 1 51097EED
 P 7250 3200
@@
 $EndComp
 $Comp
-L NPN_BCE Q1
+L matemat_power-rescue:NPN_BCE Q1
 U 1 1 510F03EF
 P 8050 2550
@@
 $EndComp
 $Comp
-L R R4
+L matemat_power-rescue:R R4
 U 1 1 510F0716
 P 7650 2250
@@
 $EndComp
 $Comp
-L R R3
+L matemat_power-rescue:R R3
 U 1 1 510F0739
 P 7650 1700
@@
 $EndComp
 $Comp
-L BZX84CSMD D12
+L matemat_power-rescue:BZX84CSMD D12
 U 1 1 510F226A
 P 7650 3450
@@
 	2400 6250 2400 6150
 Wire Wire Line
-	2800 7500 3000 7500
+	2800 7500 2950 7500
 Wire Wire Line
 	2300 7500 2300 7400
 Wire Wire Line
-	1900 7400 3000 7400
+	1900 7400 2300 7400
 Wire Wire Line
 	2800 7650 2950 7650
@@
 	1000 5000 1450 5000
 Wire Wire Line
-	1450 4950 1450 5050
+	1450 4950 1450 5000
 Connection ~ 1450 5000
 Wire Wire Line
@@
 	1000 5700 1450 5700
 Wire Wire Line
-	1450 5650 1450 5750
+	1450 5650 1450 5700
 Connection ~ 1450 5700
 Wire Wire Line
@@
 	5350 6050 5800 6050
 Wire Wire Line
-	5800 6000 5800 6100
+	5800 6000 5800 6050
 Connection ~ 5800 6050
 Wire Wire Line
@@
 	5350 6750 5800 6750
 Wire Wire Line
-	5800 6700 5800 6800
+	5800 6700 5800 6750
 Connection ~ 5800 6750
 Wire Wire Line
@@
 	6250 2850 6750 2850
 Wire Wire Line
-	6750 2800 6750 3000
+	6750 2800 6750 2850
 Connection ~ 6750 2850
 Wire Wire Line
-	7250 2800 7250 3000
+	7250 2800 7250 2950
 Wire Wire Line
 	7250 2950 6250 2950
@@
 	6750 3400 6750 3600
 Wire Wire Line
-	6750 3600 8150 3600
+	6750 3600 7250 3600
 Wire Wire Line
 	7250 3600 7250 3400
@@
 	6750 2200 7250 2200
 Wire Wire Line
-	7250 1400 7250 2400
-Wire Wire Line
-	7250 1400 8150 1400
+	7250 1400 7250 2200
+Wire Wire Line
+	7250 1400 7650 1400
 Connection ~ 7250 2200
 Wire Wire Line
@@
 Connection ~ 7650 3600
 Wire Wire Line
-	8850 2600 8850 2850
+	8850 2600 8850 2700
 Wire Wire Line
 	8850 3050 8850 3600
@@
 Connection ~ 8850 2700
 $Comp
-L +5V #PWR19
+L matemat_power-rescue:+5V #PWR19
 U 1 1 510F3CB2
 P 9050 2000
@@
 $EndComp
 $Comp
-L GND #PWR18
+L matemat_power-rescue:GND #PWR18
 U 1 1 510F3E20
 P 8850 3600
@@
 Connection ~ 7650 2550
 Wire Wire Line
-	7650 2500 7650 3350
+	7650 2500 7650 2550
 Text GLabel 6150 3650 0    60   Input ~ 0
 GNDPWR2
@@
 Wire Wire Line
 	8150 3050 8150 3100
+Wire Wire Line
+	2950 7500 3000 7500
+Wire Wire Line
+	2300 7400 3000 7400
+Wire Wire Line
+	1450 5000 1450 5050
+Wire Wire Line
+	1450 5700 1450 5750
+Wire Wire Line
+	5800 6050 5800 6100
+Wire Wire Line
+	5800 6750 5800 6800
+Wire Wire Line
+	6750 2850 6750 3000
+Wire Wire Line
+	7250 2950 7250 3000
+Wire Wire Line
+	7250 2200 7250 2400
+Wire Wire Line
+	7650 1400 8150 1400
+Wire Wire Line
+	7250 3600 7650 3600
+Wire Wire Line
+	7650 3600 8150 3600
+Wire Wire Line
+	8850 2700 8850 2850
+Wire Wire Line
+	7650 2550 7650 3350
 $EndSCHEMATC

Commit message: Recreated rescue library
Parts:
- C3, C4: symbol matemat_power-rescue:C -> matemat_power-rescue:C-matemat_power-rescue
- D10, D11, D6, D9: symbol matemat_power-rescue:DIODE -> matemat_power-rescue:DIODE-matemat_power-rescue
- D12: symbol matemat_power-rescue:BZX84CSMD -> matemat_power-rescue:BZX84CSMD-matemat_power-rescue
- IC1, IC2: symbol matemat_power-rescue:4094D -> matemat_power-rescue:4094D-matemat_power-rescue
- IC3: symbol matemat_power-rescue:ULN2803A -> matemat_power-rescue:ULN2803A-matemat_power-rescue
- IC4: symbol matemat_power-rescue:PC817 -> matemat_power-rescue:PC817-matemat_power-rescue
- J11: symbol matemat_power-rescue:CONN_8 -> matemat_power-rescue:CONN_8-matemat_power-rescue
- J4: symbol matemat:Bus_I2C -> matemat_power-rescue:Bus_I2C-matemat
- JMP1, JMP2, R1, R2, R3, R4, R5, R6: symbol matemat_power-rescue:R -> matemat_power-rescue:R-matemat_power-rescue
- Q1: symbol matemat_power-rescue:NPN_BCE -> matemat_power-rescue:NPN_BCE-matemat_power-rescue
Changed lines of the file:
@@
 EESchema Schematic File Version 4
-LIBS:matemat_power-cache
-EELAYER 26 0
+EELAYER 30 0
 EELAYER END
 $Descr A4 11693 8268
@@
 $EndDescr
 $Comp
-L matemat_power-rescue:+12V #PWR11
+L matemat_power-rescue:+12V-matemat_power-rescue #PWR11
 U 1 1 50F5F502
 P 4550 6900
@@
 $EndComp
 $Comp
-L matemat_power-rescue:+5V #PWR10
+L matemat_power-rescue:+5V-matemat_power-rescue #PWR10
 U 1 1 50F5F508
 P 2850 6800
@@
 $EndComp
 $Comp
-L matemat_power-rescue:GND #PWR12
+L matemat_power-rescue:GND-matemat_power-rescue #PWR12
 U 1 1 50F5F50E
 P 4600 6800
@@
 $EndComp
 $Comp
-L matemat:Bus_I2C J4
+L matemat_power-rescue:Bus_I2C-matemat J4
 U 1 1 50F5F5BF
 P 3650 7150
@@
 $EndComp
 $Comp
-L matemat_power-rescue:4094D IC1
+L matemat_power-rescue:4094D-matemat_power-rescue IC1
 U 1 1 50F5F7F4
 P 2600 5550
@@
 strobe
 $Comp
-L matemat_power-rescue:R JMP1
+L matemat_power-rescue:R-matemat_power-rescue JMP1
 U 1 1 50F5F6F8
 P 2550 7500
@@
 $EndComp
 $Comp
-L matemat_power-rescue:+5V #PWR9
+L matemat_power-rescue:+5V-matemat_power-rescue #PWR9
 U 1 1 50F5FA42
 P 2400 6250
@@
 $EndComp
 $Comp
-L matemat_power-rescue:R JMP2
+L matemat_power-rescue:R-matemat_power-rescue JMP2
 U 1 1 50F5FB5C
 P 2550 7650
@@
 $EndSheet
 $Comp
-L matemat_power-rescue:+5V #PWR5
+L matemat_power-rescue:+5V-matemat_power-rescue #PWR5
 U 1 1 50FF3F43
 P 1450 4950
@@
 $EndComp
 $Comp
-L matemat_power-rescue:4094D IC1
+L matemat_power-rescue:4094D-matemat_power-rescue IC1
 U 2 1 5105769F
 P 1450 5350
@@
 $EndComp
 $Comp
-L matemat_power-rescue:C C3
+L matemat_power-rescue:C-matemat_power-rescue C3
 U 1 1 510583BD
 P 1000 5300
@@
 $EndComp
 $Comp
-L matemat_power-rescue:GND #PWR6
+L matemat_power-rescue:GND-matemat_power-rescue #PWR6
 U 1 1 5105853A
 P 1450 5750
@@
 $EndComp
 $Comp
-L matemat_power-rescue:4094D IC2
+L matemat_power-rescue:4094D-matemat_power-rescue IC2
 U 1 1 510836A5
 P 6800 6350
@@
 $EndComp
 $Comp
-L matemat_power-rescue:ULN2803A IC3
+L matemat_power-rescue:ULN2803A-matemat_power-rescue IC3
 U 1 1 51086ED4
 P 8350 5150
@@
 $EndComp
 $Comp
-L matemat_power-rescue:+5V #PWR13
+L matemat_power-rescue:+5V-matemat_power-rescue #PWR13
 U 1 1 510872E7
 P 5800 6000
@@
 $EndComp
 $Comp
-L matemat_power-rescue:4094D IC2
+L matemat_power-rescue:4094D-matemat_power-rescue IC2
 U 2 1 510872ED
 P 5800 6400
@@
 $EndComp
 $Comp
-L matemat_power-rescue:C C4
+L matemat_power-rescue:C-matemat_power-rescue C4
 U 1 1 510872F3
 P 5350 6350
@@
 $EndComp
 $Comp
-L matemat_power-rescue:GND #PWR14
+L matemat_power-rescue:GND-matemat_power-rescue #PWR14
 U 1 1 51087300
 P 5800 6800
@@
 strobe
 $Comp
-L matemat_power-rescue:+5V #PWR16
+L matemat_power-rescue:+5V-matemat_power-rescue #PWR16
 U 1 1 51088412
 P 6600 7050
@@
 Dout1_Din2
 $Comp
-L matemat_power-rescue:GND #PWR17
+L matemat_power-rescue:GND-matemat_power-rescue #PWR17
 U 1 1 510888ED
 P 7850 5800
@@
 $EndComp
 $Comp
-L matemat_power-rescue:CONN_8 J11
+L matemat_power-rescue:CONN_8-matemat_power-rescue J11
 U 1 1 5108C0AA
 P 9600 5100
@@
 $EndComp
 $Comp
-L matemat_power-rescue:+12V #PWR20
+L matemat_power-rescue:+12V-matemat_power-rescue #PWR20
 U 1 1 5108D085
 P 9100 5800
@@
 $EndComp
 $Comp
-L matemat_power-rescue:R R1
+L matemat_power-rescue:R-matemat_power-rescue R1
 U 1 1 5108F808
 P 2250 7000
@@
 $EndComp
 $Comp
-L matemat_power-rescue:R R2
+L matemat_power-rescue:R-matemat_power-rescue R2
 U 1 1 5108FCDB
 P 2250 7100
@@
 $EndComp
 $Comp
-L matemat_power-rescue:+5V #PWR7
+L matemat_power-rescue:+5V-matemat_power-rescue #PWR7
 U 1 1 5108FE16
 P 1750 7000
@@
 $EndComp
 $Comp
-L matemat_power-rescue:+5V #PWR8
+L matemat_power-rescue:+5V-matemat_power-rescue #PWR8
 U 1 1 5108FE1C
 P 1750 7100
@@
 $EndComp
 $Comp
-L matemat_power-rescue:R R5
+L matemat_power-rescue:R-matemat_power-rescue R5
 U 1 1 51093461
 P 8150 3350
@@
 $EndComp
 $Comp
-L matemat_power-rescue:HT #PWR15
+L matemat_power-rescue:HT-matemat_power-rescue #PWR15
 U 1 1 51093496
 P 6250 2300
@@
 $EndComp
 $Comp
-L matemat_power-rescue:PC817 IC4
+L matemat_power-rescue:PC817-matemat_power-rescue IC4
 U 1 1 510964E4
 P 8500 2950
@@
 $EndComp
 $Comp
-L matemat_power-rescue:R R6
+L matemat_power-rescue:R-matemat_power-rescue R6
 U 1 1 51096DB7
 P 8850 2350
@@
 $EndComp
 $Comp
-L matemat_power-rescue:DIODE D6
+L matemat_power-rescue:DIODE-matemat_power-rescue D6
 U 1 1 51097ED5
 P 6750 2600
@@
 $EndComp
 $Comp
-L matemat_power-rescue:DIODE D9
+L matemat_power-rescue:DIODE-matemat_power-rescue D9
 U 1 1 51097EDD
 P 6750 3200
@@
 $EndComp
 $Comp
-L matemat_power-rescue:DIODE D10
+L matemat_power-rescue:DIODE-matemat_power-rescue D10
 U 1 1 51097EE5
 P 7250 2600
@@
 $EndComp
 $Comp
-L matemat_power-rescue:DIODE D11
+L matemat_power-rescue:DIODE-matemat_power-rescue D11
 U 1 1 51097EED
 P 7250 3200
@@
 $EndComp
 $Comp
-L matemat_power-rescue:NPN_BCE Q1
+L matemat_power-rescue:NPN_BCE-matemat_power-rescue Q1
 U 1 1 510F03EF
 P 8050 2550
@@
 $EndComp
 $Comp
-L matemat_power-rescue:R R4
+L matemat_power-rescue:R-matemat_power-rescue R4
 U 1 1 510F0716
 P 7650 2250
@@
 $EndComp
 $Comp
-L matemat_power-rescue:R R3
+L matemat_power-rescue:R-matemat_power-rescue R3
 U 1 1 510F0739
 P 7650 1700
@@
 $EndComp
 $Comp
-L matemat_power-rescue:BZX84CSMD D12
+L matemat_power-rescue:BZX84CSMD-matemat_power-rescue D12
 U 1 1 510F226A
 P 7650 3450
@@
 Connection ~ 8850 2700
 $Comp
-L matemat_power-rescue:+5V #PWR19
+L matemat_power-rescue:+5V-matemat_power-rescue #PWR19
 U 1 1 510F3CB2
 P 9050 2000
@@
 $EndComp
 $Comp
-L matemat_power-rescue:GND #PWR18
+L matemat_power-rescue:GND-matemat_power-rescue #PWR18
 U 1 1 510F3E20
 P 8850 3600

Commit message: Cleaned up schematics and removed obsolete parts
Parts:
- removed unit 2 of IC1
- removed unit 2 of IC2
- C3, C4: footprint SM0805 -> Capacitor_SMD:C_0805_2012Metric_Pad1.18x1.45mm_HandSolder; symbol matemat_power-rescue:C-matemat_power-rescue -> Device:C
- D10, D11, D6, D9: footprint DO214 -> Diode_SMD:D_SMA_Handsoldering; symbol matemat_power-rescue:DIODE-matemat_power-rescue -> Device:D_Schottky
- D12: footprint _sto-SOT23-DIODE -> Diode_SMD:D_SOT-23_ANK; symbol matemat_power-rescue:BZX84CSMD-matemat_power-rescue -> Device:D_Zener
- IC1, IC2: value 4094D -> 74HC4094; footprint -SO16 -> Package_SO:SOIC-16_3.9x9.9mm_P1.27mm; symbol matemat_power-rescue:4094D-matemat_power-rescue -> oni:74HC4094
- IC3: footprint -SO18-1 -> Package_SO:SOIC-18W_7.5x11.6mm_P1.27mm; symbol matemat_power-rescue:ULN2803A-matemat_power-rescue -> Transistor_Array:ULN2803A
- IC4: footprint -DIL04 -> Package_DIP:DIP-4_W7.62mm; symbol matemat_power-rescue:PC817-matemat_power-rescue -> Isolator:PC817
- J11: footprint Bornier_B8_Phoenix -> TerminalBlock_Phoenix:TerminalBlock_Phoenix_PTSM-0,5-8-2.5-H-THR_1x08_P2.50mm_Horizontal; symbol matemat_power-rescue:CONN_8-matemat_power-rescue -> Connector_Generic:Conn_01x08
- J4: footprint he10-16ds -> Connector_PinHeader_2.54mm:PinHeader_2x08_P2.54mm_Vertical; symbol matemat_power-rescue:Bus_I2C-matemat -> Connector_Generic:Conn_02x08_Odd_Even
- JMP1, JMP2, R1, R2: footprint SM0603 -> Resistor_SMD:R_0603_1608Metric_Pad0.98x0.95mm_HandSolder; symbol matemat_power-rescue:R-matemat_power-rescue -> Device:R
- Q1: footprint _sto-TO220V -> Package_TO_SOT_THT:TO-220-3_Vertical; symbol matemat_power-rescue:NPN_BCE-matemat_power-rescue -> Device:Q_NPN_BCE
- R3, R4: footprint -0309/12 -> Resistor_THT:R_Axial_DIN0309_L9.0mm_D3.2mm_P12.70mm_Horizontal; symbol matemat_power-rescue:R-matemat_power-rescue -> Device:R
- R5, R6: footprint SM0805 -> Resistor_SMD:R_0805_2012Metric_Pad1.20x1.40mm_HandSolder; symbol matemat_power-rescue:R-matemat_power-rescue -> Device:R
Connections:
- net +12V: now also R1.2, R2.2
- net +5V: now also C3.2, C4.2, IC1.16 (VCC), IC2.16 (VCC); no longer C3.1, C4.1, R1.2, R2.2
- net GND: now also C3.1, C4.1, IC1.8 (GND), IC2.8 (GND); no longer C3.2, C4.2
- net at Q1.2 (C), R3.1: now also D10.1 (K), D6.1 (K); no longer D10.2 (K), D6.2 (K)
- net at Q1.1 (B), R4.2: now also D12.1 (K); no longer D12.C
- net GNDPWR2: no longer names the net of D11.2 (A)
- net GNDPWR2: now also D12.2 (A), D9.2 (A), R5.2; no longer D10.1 (A)
- removed net HT: D6.1 (A), D9.2 (K)
- new net AC: D10.2 (A), D11.1 (K)
- new net LINE: D6.2 (A), D9.1 (K)
Other:
- moved on the sheet: C3, C4, JMP1, JMP2, R1, R2

Commit message: Updated PCB layout
Parts:
- J11: footprint TerminalBlock_Phoenix:TerminalBlock_Phoenix_PTSM-0,5-8-2.5-H-THR_1x08_P2.50mm_Horizontal -> TerminalBlock_Phoenix:TerminalBlock_Phoenix_MPT-0,5-8-2.54_1x08_P2.54mm_Horizontal

Commit message: Replaced power board diode pad layouts
Parts:
- D10, D11, D6, D9: footprint Diode_SMD:D_SMA_Handsoldering -> Diode_SMD:D_SMA
Changed lines of the file:
@@
 F 0 "D6" H 6750 2700 40  0000 C CNN
 F 1 "CDBA2100-G" H 6750 2500 40  0000 C CNN
-F 2 "Diode_SMD:D_SMA_Handsoldering" H 6750 2600 60  0001 C CNN
+F 2 "Diode_SMD:D_SMA" H 6750 2600 60  0001 C CNN
 F 3 "" H 6750 2600 60  0001 C CNN
 F 4 "RS 636-5088" H 6750 2600 60  0001 C CNN "Reference"
@@
 F 0 "D9" H 6750 3300 40  0000 C CNN
 F 1 "CDBA2100-G" H 6750 3100 40  0000 C CNN
-F 2 "Diode_SMD:D_SMA_Handsoldering" H 6750 3200 60  0001 C CNN
+F 2 "Diode_SMD:D_SMA" H 6750 3200 60  0001 C CNN
 F 3 "" H 6750 3200 60  0001 C CNN
 F 4 "RS 636-5088" H 6750 3200 60  0001 C CNN "Reference"
@@
 F 0 "D10" H 7250 2700 40  0000 C CNN
 F 1 "CDBA2100-G" H 7250 2500 40  0000 C CNN
-F 2 "Diode_SMD:D_SMA_Handsoldering" H 7250 2600 60  0001 C CNN
+F 2 "Diode_SMD:D_SMA" H 7250 2600 60  0001 C CNN
 F 3 "" H 7250 2600 60  0001 C CNN
 F 4 "RS 636-5088" H 7250 2600 60  0001 C CNN "Reference"
@@
 F 0 "D11" H 7250 3300 40  0000 C CNN
 F 1 "CDBA2100-G" H 7250 3100 40  0000 C CNN
-F 2 "Diode_SMD:D_SMA_Handsoldering" H 7250 3200 60  0001 C CNN
+F 2 "Diode_SMD:D_SMA" H 7250 3200 60  0001 C CNN
 F 3 "" H 7250 3200 60  0001 C CNN
 F 4 "RS 636-5088" H 7250 3200 60  0001 C CNN "Reference"
